File: vlf_receiver.kicad_pcb (KiCad board)
At the start: 2 copper layers, 4 parts, among them U1 LMP7721, U2 TLE2426xLP

Commit message: Update.
Parts:
- added J1: OUT, TerminalBlock_RND:TerminalBlock_RND_205-00001_1x02_P5.00mm_Horizontal, F.Cu at (92.7, 73.7)
- added J2: ANT+, Connector_Pin:Pin_D1.0mm_L10.0mm, F.Cu at (109.2, 64.8)
- added J3: ANT-, Connector_Pin:Pin_D1.0mm_L10.0mm, F.Cu at (114.3, 64.8)
- added J4: BLEED-R, Connector_Pin:Pin_D1.0mm_L10.0mm, F.Cu at (127.0, 64.8)
- added J5: FILT-C, Connector_Pin:Pin_D1.0mm_L10.0mm, F.Cu at (120.7, 64.8)
- added J6: VCC, TerminalBlock_RND:TerminalBlock_RND_205-00001_1x02_P5.00mm_Horizontal, F.Cu at (143.5, 72.4)
Connections:
- U1 pad 1: (no net) -> Net-(J2-Pad1)
Routing:
- net Net-(R1-Pad1): track 0.00 -> 6.22 mm
