File: PCB/capacitor_square/capacitor_square/capacitor_square.kicad_pcb (KiCad board)
At the start: 2 copper layers, 15.2 x 15.2 mm, 0 parts

Commit message: Clean up capacitor_square project and gitignore KiCad artifacts
Remove unneeded schematic, symbol lib, and footprint dir from
capacitor_square (PCB-only project, no schematic needed).
Remove back silkscreen GND text. Fix KiCad S-expression syntax
(no comments, no 'justify center'). Gitignore KiCad auto-generated
files (*-backups/, *.kicad_prl, fp-info-cache) across all projects.

Co-Authored-By: Claude Opus 4.6 (1M context) <noreply@anthropic.com>
Other:
- board text removed: "GND"
Changed lines of the file:
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@@
   )
   (net 0 "")
-  ; Board outline  15.20 x 15.20 mm
   (gr_rect
     (start -7.6000 -7.6000)
@@
     (layer "Edge.Cuts")
   )
-  ; Top capacitor plate  14.20 x 14.20 mm (pullback 0.50 mm)
   (gr_rect
     (start -7.1000 -7.1000)
@@
     (layer "F.Cu")
   )
-  ; Bottom capacitor plate  14.20 x 14.20 mm
   (gr_rect
     (start -7.1000 -7.1000)
@@
     (layer "B.Cu")
   )
-  ; Top solder mask opening  2.0 x 2.0 mm (wire attachment point)
   (gr_rect
     (start -1.0000 -1.0000)
@@
     (layer "F.Mask")
   )
-  ; Bottom solder mask opening  2.0 x 2.0 mm
   (gr_rect
     (start -1.0000 -1.0000)
@@
     (layer "B.Mask")
   )
-  ; Front silkscreen  capacitor value and project
   (gr_text "ELARA"
     (at 0 -5.9000)
@@
     (effects
       (font (size 1.20 1.20) (thickness 0.180))
-      (justify center)
     )
   )
@@
     (effects
       (font (size 1.20 1.20) (thickness 0.180))
-      (justify center)
     )
   )
-  ; Back silkscreen
-  (gr_text "GND"
-    (at 0 0)
-    (layer "B.SilkS")
-    (effects
-      (font (size 1.20 1.20) (thickness 0.180))
-      (justify center mirror)
-    )
-  )
-  ; Fabrication notes
   (gr_text "15.20 x 15.20 mm, FR4 0.80 mm, 10.0pF"
     (at 0 9.6000)
@@
     (effects
       (font (size 1.0 1.0) (thickness 0.15))
-      (justify center)
     )
   )
-  ; Courtyard
   (gr_rect
     (start -7.8500 -7.8500)
