File: PCB/antenna_amplifier/antenna_amplifier.kicad_sch (KiCad schematic)
At the start: 34 parts, among them J1 ANT_IN, J2 SPDIF_COAX, J3 PWR_IN, J4 ANT_BIAS, J5 AES_EBU, U1 LMP7721, U2 LMP7715, U3 PCM1804, U4 CS8406, U5 ADM7150-5.0, U6 ADM7150-3.3, U7 LMP7715, Y1 24.576MHz

Commit message: Add kicad_wirer tool, complete PCM1804 wiring
New tool: tools/kicad_wirer.py — parses KiCad schematics,
computes absolute pin positions from lib_symbols + placement
transforms, and checks connectivity. Use --report for pin
positions, --connectivity for unconnected pin detection.

PCM1804 wiring completed:
  - Pin 15 (DATA) → DOUT label to CS8406
  - Pin 16 (BCK) → BCK label to CS8406
  - Pin 19 (RST) → +3V3D pullup
  - Pin 6 (FMT0) → +3V3D (I2S format)
  - Pins 7,8 (FMT1, S/M) → GND bus (I2S, master mode)
  - Pins 9-11 (OSR0-2) → GND bus (quad rate 192kHz)
  - Pin 22 (VCC) → +5VA
  - Pins 2,27 (AGNDL,AGNDR) → GND
  - Pins 20,21 (OVFL,OVFR) → no-connect

Connectivity check: U3 has 27/28 pins connected (OVFR is
intentional no-connect).

Co-Authored-By: Claude Opus 4.6 (1M context) <noreply@anthropic.com>
Connections:
- net +3V3D: now also U3.19 (RST), U3.6 (FMT0)
- net +5VA: now also U3.10 (OSR1), U3.11 (OSR2), U3.2 (AGNDL), U3.22 (VCC), U3.27 (AGNDR), U3.7 (FMT1), U3.8 (S/M), U3.9 (OSR0)
- net BCK: now also U3.16 (BCK)
- net DOUT: now also U3.15 (DATA)
- no-connect marks 1 -> 3
Changed lines of the file:
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@@
 	(wire (pts (xy 210.82 71.12) (xy 218.44 71.12))
 		(stroke (width 0) (type solid)))
+	(wire (pts (xy 243.84 66.04) (xy 248.92 66.04))
+		(stroke (width 0) (type solid)))
+	(label "DOUT" (at 248.92 66.04 0)
+		(effects (font (size 1.27 1.27))))
+	(wire (pts (xy 243.84 68.58) (xy 248.92 68.58))
+		(stroke (width 0) (type solid)))
+	(label "BCK" (at 248.92 68.58 0)
+		(effects (font (size 1.27 1.27))))
+	(wire (pts (xy 243.84 78.74) (xy 248.92 78.74))
+		(stroke (width 0) (type solid)))
+	(wire (pts (xy 248.92 78.74) (xy 248.92 73.66))
+		(stroke (width 0) (type solid)))
+	(symbol
+		(lib_id "power:+3V3D")
+		(at 248.92 73.66 0)
+		(unit 1)
+		(exclude_from_sim no) (in_bom yes) (on_board yes) (dnp no)
+		(property "Reference" "#PWR91" (at 248.92 71.66 0) (effects (font (size 1.27 1.27)) (hide yes)))
+		(property "Value" "+3V3D" (at 248.92 69.85 0) (effects (font (size 1.27 1.27))))
+		(instances (project "antenna_amplifier"
+			(path "/09f45598-3e76-49a4-ba12-a3a92a2874f1" (reference "#PWR91") (unit 1)))))
+	(no_connect (at 243.84 83.82))
+	(no_connect (at 243.84 81.28))
+	(wire (pts (xy 243.84 88.9) (xy 248.92 88.9))
+		(stroke (width 0) (type solid)))
+	(wire (pts (xy 248.92 88.9) (xy 248.92 83.82))
+		(stroke (width 0) (type solid)))
+	(symbol
+		(lib_id "power:+3V3D")
+		(at 248.92 83.82 0)
+		(unit 1)
+		(exclude_from_sim no) (in_bom yes) (on_board yes) (dnp no)
+		(property "Reference" "#PWR92" (at 248.92 81.82 0) (effects (font (size 1.27 1.27)) (hide yes)))
+		(property "Value" "+3V3D" (at 248.92 80.01 0) (effects (font (size 1.27 1.27))))
+		(instances (project "antenna_amplifier"
+			(path "/09f45598-3e76-49a4-ba12-a3a92a2874f1" (reference "#PWR92") (unit 1)))))
+	(wire (pts (xy 243.84 91.44) (xy 253.99 91.44))
+		(stroke (width 0) (type solid)))
+	(wire (pts (xy 243.84 93.98) (xy 253.99 93.98))
+		(stroke (width 0) (type solid)))
+	(wire (pts (xy 243.84 96.52) (xy 253.99 96.52))
+		(stroke (width 0) (type solid)))
+	(wire (pts (xy 243.84 99.06) (xy 253.99 99.06))
+		(stroke (width 0) (type solid)))
+	(wire (pts (xy 243.84 101.6) (xy 253.99 101.6))
+		(stroke (width 0) (type solid)))
+	(wire (pts (xy 253.99 91.44) (xy 253.99 93.98))
+		(stroke (width 0) (type solid)))
+	(wire (pts (xy 253.99 93.98) (xy 253.99 96.52))
+		(stroke (width 0) (type solid)))
+	(wire (pts (xy 253.99 96.52) (xy 253.99 99.06))
+		(stroke (width 0) (type solid)))
+	(wire (pts (xy 253.99 99.06) (xy 253.99 101.6))
+		(stroke (width 0) (type solid)))
+	(wire (pts (xy 253.99 101.6) (xy 253.99 106.68))
+		(stroke (width 0) (type solid)))
+	(symbol
+		(lib_id "power:GND")
+		(at 253.99 106.68 0)
+		(unit 1)
+		(exclude_from_sim no) (in_bom yes) (on_board yes) (dnp no)
+		(property "Reference" "#PWR93" (at 253.99 104.68 0) (effects (font (size 1.27 1.27)) (hide yes)))
+		(property "Value" "GND" (at 253.99 109.68 0) (effects (font (size 1.27 1.27))))
+		(instances (project "antenna_amplifier"
+			(path "/09f45598-3e76-49a4-ba12-a3a92a2874f1" (reference "#PWR93") (unit 1)))))
+	(wire (pts (xy 226.06 59.69) (xy 226.06 54.61))
+		(stroke (width 0) (type solid)))
+	(symbol
+		(lib_id "power:+5VA")
+		(at 226.06 54.61 0)
+		(unit 1)
+		(exclude_from_sim no) (in_bom yes) (on_board yes) (dnp no)
+		(property "Reference" "#PWR94" (at 226.06 52.61 0) (effects (font (size 1.27 1.27)) (hide yes)))
+		(property "Value" "+5VA" (at 226.06 50.8 0) (effects (font (size 1.27 1.27))))
+		(instances (project "antenna_amplifier"
+			(path "/09f45598-3e76-49a4-ba12-a3a92a2874f1" (reference "#PWR94") (unit 1)))))
+	(wire (pts (xy 220.98 107.95) (xy 220.98 113.03))
+		(stroke (width 0) (type solid)))
+	(symbol
+		(lib_id "power:GND")
+		(at 220.98 113.03 0)
+		(unit 1)
+		(exclude_from_sim no) (in_bom yes) (on_board yes) (dnp no)
+		(property "Reference" "#PWR95" (at 220.98 111.03 0) (effects (font (size 1.27 1.27)) (hide yes)))
+		(property "Value" "GND" (at 220.98 116.03 0) (effects (font (size 1.27 1.27))))
+		(instances (project "antenna_amplifier"
+			(path "/09f45598-3e76-49a4-ba12-a3a92a2874f1" (reference "#PWR95") (unit 1)))))
+	(wire (pts (xy 236.22 107.95) (xy 236.22 113.03))
+		(stroke (width 0) (type solid)))
+	(symbol
+		(lib_id "power:GND")
+		(at 236.22 113.03 0)
+		(unit 1)
+		(exclude_from_sim no) (in_bom yes) (on_board yes) (dnp no)
+		(property "Reference" "#PWR96" (at 236.22 111.03 0) (effects (font (size 1.27 1.27)) (hide yes)))
+		(property "Value" "GND" (at 236.22 116.03 0) (effects (font (size 1.27 1.27))))
+		(instances (project "antenna_amplifier"
+			(path "/09f45598-3e76-49a4-ba12-a3a92a2874f1" (reference "#PWR96") (unit 1)))))
 	(no_connect
 		(at 147.32 81.28)

Commit message: Set preamp gain to 40 dB (Rf=100k, Cf=15nF)
The maximum amplification is dictated by 50 Hz mains E-field
pickup. With the LMP7721's 1 Tohm input impedance and 6.5m
effective antenna height, a power line at 100m produces ~1-5 mV
of 50 Hz at the antenna. 40 dB (100x) keeps this within the
ADC's linear range (25 mV max input before clipping, 73 dB
headroom). The 50 Hz is removed cleanly by a digital notch
filter in software.

Rf=100k, Cf=15nF (C0G), Rg=1k, Cg=100uF.
G = 101 (40.1 dB), fc = 106 Hz.

Previous experience with Romero-like design needed 60 dB sound
card gain, but sound cards have ~10-50k input impedance which
attenuates the 50 Hz E-field. The electrometer's 1 Tohm input
picks up everything, requiring lower analog gain.

Added expected_signal.py simulation with Schumann resonance
E-field levels from published measurements (Sentman, Nickolaenko
& Hayakawa, Price & Melnikov).

Co-Authored-By: Claude Opus 4.6 (1M context) <noreply@anthropic.com>
Parts:
- Cf: value 150n -> 15n
- Rf: value 9.1k -> 100k
Changed lines of the file:
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@@
 			)
 		)
-		(property "Value" "9.1k"
+		(property "Value" "100k"
 			(at 141.7 58.88 0)
 			(effects
@@
 			)
 		)
-		(property "Value" "150n"
+		(property "Value" "15n"
 			(at 162.02 58.88 0)
 			(effects
