File: PCB/antenna_amplifier/digital.kicad_sch (KiCad schematic)
At the start: 31 parts, among them J401 AES3 OUT, J402 S/PDIF OUT, SW401 CS8406 MODE, U401 CS8406, Y401 24.576MHz

Commit message: Drop amplifier power LED, add turret and pulse-transformer footprints, start PCB generator
The amplifier board can run from a battery, so it has no power LED;
the overload LED only lights while the ADC clips. Adds PCB/elara.pretty
(PTFE input turret, DIP-6 digital-audio transformer outline -- pinout
to be verified against the Newava datasheet) and a work-in-progress
pcbnew-based layout generator.

Co-Authored-By: Claude Opus 5.5 <noreply@anthropic.com>
Claude-Session: https://claude.ai/code/session_01RsM1DhHhY1tSr2aHjVygSC
Parts:
- TR401, TR402: footprint elara:Transformer_Pulse_DIP-8_W7.62mm -> elara:Transformer_Pulse_DIP-6_W7.62mm
Changed lines of the file:
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@@
 		(on_board yes)
 		(dnp no)
-		(property "Reference" "#PWR093"
+		(property "Reference" "#PWR091"
 			(at 38.1 33.02 0)
 			(effects
@@
 			(project "antenna_amplifier"
 				(path "/61336681-2262-5f00-9d69-45832dcbe407/0ae99a2d-b679-543a-8f49-e431d07ea905"
-					(reference "#PWR093")
+					(reference "#PWR091")
 					(unit 1)
 				)
@@
 		(on_board yes)
 		(dnp no)
-		(property "Reference" "#PWR094"
+		(property "Reference" "#PWR092"
 			(at 38.1 58.42 0)
 			(effects
@@
 			(project "antenna_amplifier"
 				(path "/61336681-2262-5f00-9d69-45832dcbe407/0ae99a2d-b679-543a-8f49-e431d07ea905"
-					(reference "#PWR094")
+					(reference "#PWR092")
 					(unit 1)
 				)
@@
 		(on_board yes)
 		(dnp no)
-		(property "Reference" "#PWR095"
+		(property "Reference" "#PWR093"
 			(at 100.33 55.88 0)
 			(effects
@@
 			(project "antenna_amplifier"
 				(path "/61336681-2262-5f00-9d69-45832dcbe407/0ae99a2d-b679-543a-8f49-e431d07ea905"
-					(reference "#PWR095")
+					(reference "#PWR093")
 					(unit 1)
 				)
@@
 		(on_board yes)
 		(dnp no)
-		(property "Reference" "#PWR096"
+		(property "Reference" "#PWR094"
 			(at 100.33 68.58 0)
 			(effects
@@
 			(project "antenna_amplifier"
 				(path "/61336681-2262-5f00-9d69-45832dcbe407/0ae99a2d-b679-543a-8f49-e431d07ea905"
-					(reference "#PWR096")
+					(reference "#PWR094")
 					(unit 1)
 				)
@@
 		(on_board yes)
 		(dnp no)
-		(property "Reference" "#PWR097"
+		(property "Reference" "#PWR095"
 			(at 162.56 53.34 0)
 			(effects
@@
 			(project "antenna_amplifier"
 				(path "/61336681-2262-5f00-9d69-45832dcbe407/0ae99a2d-b679-543a-8f49-e431d07ea905"
-					(reference "#PWR097")
+					(reference "#PWR095")
 					(unit 1)
 				)
@@
 		(on_board yes)
 		(dnp no)
-		(property "Reference" "#PWR098"
+		(property "Reference" "#PWR096"
 			(at 203.2 86.36 0)
 			(effects
@@
 			(project "antenna_amplifier"
 				(path "/61336681-2262-5f00-9d69-45832dcbe407/0ae99a2d-b679-543a-8f49-e431d07ea905"
-					(reference "#PWR098")
+					(reference "#PWR096")
 					(unit 1)
 				)
@@
 		(on_board yes)
 		(dnp no)
-		(property "Reference" "#PWR099"
+		(property "Reference" "#PWR097"
 			(at 180.34 40.64 0)
 			(effects
@@
 			(project "antenna_amplifier"
 				(path "/61336681-2262-5f00-9d69-45832dcbe407/0ae99a2d-b679-543a-8f49-e431d07ea905"
-					(reference "#PWR099")
+					(reference "#PWR097")
 					(unit 1)
 				)
@@
 		(on_board yes)
 		(dnp no)
-		(property "Reference" "#PWR100"
+		(property "Reference" "#PWR098"
 			(at 182.88 96.52 0)
 			(effects
@@
 			(project "antenna_amplifier"
 				(path "/61336681-2262-5f00-9d69-45832dcbe407/0ae99a2d-b679-543a-8f49-e431d07ea905"
-					(reference "#PWR100")
+					(reference "#PWR098")
 					(unit 1)
 				)
@@
 		(on_board yes)
 		(dnp no)
-		(property "Reference" "#PWR101"
+		(property "Reference" "#PWR099"
 			(at 185.42 40.64 0)
 			(effects
@@
 			(project "antenna_amplifier"
 				(path "/61336681-2262-5f00-9d69-45832dcbe407/0ae99a2d-b679-543a-8f49-e431d07ea905"
-					(reference "#PWR101")
+					(reference "#PWR099")
 					(unit 1)
 				)
@@
 		(on_board yes)
 		(dnp no)
-		(property "Reference" "#PWR102"
+		(property "Reference" "#PWR100"
 			(at 124.46 118.11 0)
 			(effects
@@
 			(project "antenna_amplifier"
 				(path "/61336681-2262-5f00-9d69-45832dcbe407/0ae99a2d-b679-543a-8f49-e431d07ea905"
-					(reference "#PWR102")
+					(reference "#PWR100")
 					(unit 1)
 				)
@@
 		(on_board yes)
 		(dnp no)
-		(property "Reference" "#PWR103"
+		(property "Reference" "#PWR101"
 			(at 207.01 105.41 0)
 			(effects
@@
 			(project "antenna_amplifier"
 				(path "/61336681-2262-5f00-9d69-45832dcbe407/0ae99a2d-b679-543a-8f49-e431d07ea905"
-					(reference "#PWR103")
+					(reference "#PWR101")
 					(unit 1)
 				)
@@
 		(on_board yes)
 		(dnp no)
-		(property "Reference" "#PWR104"
+		(property "Reference" "#PWR102"
 			(at 207.01 118.11 0)
 			(effects
@@
 			(project "antenna_amplifier"
 				(path "/61336681-2262-5f00-9d69-45832dcbe407/0ae99a2d-b679-543a-8f49-e431d07ea905"
-					(reference "#PWR104")
+					(reference "#PWR102")
 					(unit 1)
 				)
@@
 		(on_board yes)
 		(dnp no)
-		(property "Reference" "#PWR105"
+		(property "Reference" "#PWR103"
 			(at 219.71 105.41 0)
 			(effects
@@
 			(project "antenna_amplifier"
 				(path "/61336681-2262-5f00-9d69-45832dcbe407/0ae99a2d-b679-543a-8f49-e431d07ea905"
-					(reference "#PWR105")
+					(reference "#PWR103")
 					(unit 1)
 				)
@@
 		(on_board yes)
 		(dnp no)
-		(property "Reference" "#PWR106"
+		(property "Reference" "#PWR104"
 			(at 219.71 118.11 0)
 			(effects
@@
 			(project "antenna_amplifier"
 				(path "/61336681-2262-5f00-9d69-45832dcbe407/0ae99a2d-b679-543a-8f49-e431d07ea905"
-					(reference "#PWR106")
+					(reference "#PWR104")
 					(unit 1)
 				)
@@
 		(on_board yes)
 		(dnp no)
-		(property "Reference" "#PWR107"
+		(property "Reference" "#PWR105"
 			(at 232.41 105.41 0)
 			(effects
@@
 			(project "antenna_amplifier"
 				(path "/61336681-2262-5f00-9d69-45832dcbe407/0ae99a2d-b679-543a-8f49-e431d07ea905"
-					(reference "#PWR107")
+					(reference "#PWR105")
 					(unit 1)
 				)
@@
 		(on_board yes)
 		(dnp no)
-		(property "Reference" "#PWR108"
+		(property "Reference" "#PWR106"
 			(at 232.41 118.11 0)
 			(effects
@@
 			(project "antenna_amplifier"
 				(path "/61336681-2262-5f00-9d69-45832dcbe407/0ae99a2d-b679-543a-8f49-e431d07ea905"
-					(reference "#PWR108")
+					(reference "#PWR106")
 					(unit 1)
 				)
@@
 		(on_board yes)
 		(dnp no)
-		(property "Reference" "#PWR109"
+		(property "Reference" "#PWR107"
 			(at 265.43 35.56 0)
 			(effects
@@
 			(project "antenna_amplifier"
 				(path "/61336681-2262-5f00-9d69-45832dcbe407/0ae99a2d-b679-543a-8f49-e431d07ea905"
-					(reference "#PWR109")
+					(reference "#PWR107")
 					(unit 1)
 				)
@@
 		(on_board yes)
 		(dnp no)
-		(property "Reference" "#PWR110"
+		(property "Reference" "#PWR108"
 			(at 308.61 57.15 0)
 			(effects
@@
 			(project "antenna_amplifier"
 				(path "/61336681-2262-5f00-9d69-45832dcbe407/0ae99a2d-b679-543a-8f49-e431d07ea905"
-					(reference "#PWR110")
+					(reference "#PWR108")
 					(unit 1)
 				)
@@
 		(on_board yes)
 		(dnp no)
-		(property "Reference" "#PWR111"
+		(property "Reference" "#PWR109"
 			(at 320.04 57.15 0)
 			(effects
@@
 			(project "antenna_amplifier"
 				(path "/61336681-2262-5f00-9d69-45832dcbe407/0ae99a2d-b679-543a-8f49-e431d07ea905"
-					(reference "#PWR111")
+					(reference "#PWR109")
 					(unit 1)
 				)
@@
 		(on_board yes)
 		(dnp no)
-		(property "Reference" "#PWR112"
+		(property "Reference" "#PWR110"
 			(at 331.47 57.15 0)
 			(effects
@@
 			(project "antenna_amplifier"
 				(path "/61336681-2262-5f00-9d69-45832dcbe407/0ae99a2d-b679-543a-8f49-e431d07ea905"
-					(reference "#PWR112")
+					(reference "#PWR110")
 					(unit 1)
 				)
@@
 		(on_board yes)
 		(dnp no)
-		(property "Reference" "#PWR113"
+		(property "Reference" "#PWR111"
 			(at 342.9 57.15 0)
 			(effects
@@
 			(project "antenna_amplifier"
 				(path "/61336681-2262-5f00-9d69-45832dcbe407/0ae99a2d-b679-543a-8f49-e431d07ea905"
-					(reference "#PWR113")
+					(reference "#PWR111")
 					(unit 1)
 				)
@@
 		(on_board yes)
 		(dnp no)
-		(property "Reference" "#PWR114"
+		(property "Reference" "#PWR112"
 			(at 354.33 57.15 0)
 			(effects
@@
 			(project "antenna_amplifier"
 				(path "/61336681-2262-5f00-9d69-45832dcbe407/0ae99a2d-b679-543a-8f49-e431d07ea905"
-					(reference "#PWR114")
+					(reference "#PWR112")
 					(unit 1)
 				)
@@
 		(on_board yes)
 		(dnp no)
-		(property "Reference" "#PWR115"
+		(property "Reference" "#PWR113"
 			(at 365.76 57.15 0)
 			(effects
@@
 			(project "antenna_amplifier"
 				(path "/61336681-2262-5f00-9d69-45832dcbe407/0ae99a2d-b679-543a-8f49-e431d07ea905"
-					(reference "#PWR115")
+					(reference "#PWR113")
 					(unit 1)
 				)
@@
 		(on_board yes)
 		(dnp no)
-		(property "Reference" "#PWR116"
+		(property "Reference" "#PWR114"
 			(at 377.19 57.15 0)
 			(effects
@@
 			(project "antenna_amplifier"
 				(path "/61336681-2262-5f00-9d69-45832dcbe407/0ae99a2d-b679-543a-8f49-e431d07ea905"
-					(reference "#PWR116")
+					(reference "#PWR114")
 					(unit 1)
 				)
@@
 		(on_board yes)
 		(dnp no)
-		(property "Reference" "#PWR117"
+		(property "Reference" "#PWR115"
 			(at 388.62 57.15 0)
 			(effects
@@
 			(project "antenna_amplifier"
 				(path "/61336681-2262-5f00-9d69-45832dcbe407/0ae99a2d-b679-543a-8f49-e431d07ea905"
-					(reference "#PWR117")
+					(reference "#PWR115")
 					(unit 1)
 				)
@@
 			)
 		)
-		(property "Footprint" "elara:Transformer_Pulse_DIP-8_W7.62mm"
+		(property "Footprint" "elara:Transformer_Pulse_DIP-6_W7.62mm"
 			(at 99.06 160.02 0)
 			(effects
@@
 		(on_board yes)
 		(dnp no)
-		(property "Reference" "#PWR118"
+		(property "Reference" "#PWR116"
 			(at 152.4 179.07 0)
 			(effects
@@
 			(project "antenna_amplifier"
 				(path "/61336681-2262-5f00-9d69-45832dcbe407/0ae99a2d-b679-543a-8f49-e431d07ea905"
-					(reference "#PWR118")
+					(reference "#PWR116")
 					(unit 1)
 				)
@@
 		(on_board yes)
 		(dnp no)
-		(property "Reference" "#PWR119"
+		(property "Reference" "#PWR117"
 			(at 165.1 179.07 0)
 			(effects
@@
 			(project "antenna_amplifier"
 				(path "/61336681-2262-5f00-9d69-45832dcbe407/0ae99a2d-b679-543a-8f49-e431d07ea905"
-					(reference "#PWR119")
+					(reference "#PWR117")
 					(unit 1)
 				)
@@
 			)
 		)
-		(property "Footprint" "elara:Transformer_Pulse_DIP-8_W7.62mm"
+		(property "Footprint" "elara:Transformer_Pulse_DIP-6_W7.62mm"
 			(at 302.26 160.02 0)
 			(effects

Commit message: Route the two-bucket PSU board: fully connected, DRC clean but one thermal
Freerouting 1.9 in batch mode (2.1 never saved its session). Grounds
are routed on this board because the relays switch bucket current in
the unpoured area; mains nets 1.0 mm / 2.0 mm, current paths 0.6 mm;
hand-routed 1 mm PE rail on the left edge, GND_C-PE bond at the PE
hole; only the two mains-side holes are PE, the receiver-side holes
are unplated. Plain exposed-pad footprints (the thermal-via variants
need 0.2 mm drills). Newava S2208x redrawn as a 4-pin part (windings
1-2 / 3-4 per the DCR spec) with slotted pins 2/4 fitting either pitch.

Co-Authored-By: Claude Opus 5.5 <noreply@anthropic.com>
Claude-Session: https://claude.ai/code/session_01RsM1DhHhY1tSr2aHjVygSC
Parts:
- TR401, TR402: footprint elara:Transformer_Pulse_DIP-6_W7.62mm -> elara:Transformer_Pulse_4Pin_W7.62mm
Changed lines of the file:
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@@
 			)
 		)
-		(property "Footprint" "elara:Transformer_Pulse_DIP-6_W7.62mm"
+		(property "Footprint" "elara:Transformer_Pulse_4Pin_W7.62mm"
 			(at 99.06 160.02 0)
 			(effects
@@
 			)
 		)
-		(property "Description" "AES3 110 R pulse transformer 1:1 (verify pinout vs footprint)"
+		(property "Description" "AES3 110 R pulse transformer 1:1 (4-pin, windings 1-2 / 3-4; slots fit 5.08 or 10.16 mm pitch)"
 			(at 99.06 160.02 0)
 			(effects
@@
 			)
 		)
-		(property "Footprint" "elara:Transformer_Pulse_DIP-6_W7.62mm"
+		(property "Footprint" "elara:Transformer_Pulse_4Pin_W7.62mm"
 			(at 302.26 160.02 0)
 			(effects
@@
 			)
 		)
-		(property "Description" "S/PDIF 75 R pulse transformer 1:1 (verify pinout vs footprint)"
+		(property "Description" "S/PDIF 75 R pulse transformer 1:1 (4-pin, windings 1-2 / 3-4; slots fit 5.08 or 10.16 mm pitch)"
 			(at 302.26 160.02 0)
 			(effects

Commit message: Apply simulation fixes; add PSU/stability/system sims and priced BOM
simulations/psu: the charger caps each bucket at ~10.3 V, so the LT3045
at 8.45 V dropped out. Now R_SET 69.8k (6.98 V) and a 15 s swap
(CD4060 Rt 80.6k): +1.97 V headroom nominal, +0.49 V worst corner.
Charger output cap 10 uF -> 100 nF (3 A cold-start contact spike).
Swap artefact >= 83 dB below the floor; 50 Hz leakage 4-5 orders lower
than a direct AC-DC module (earth the receiver ground locally).
simulations/stability: guard buffer U202 had 43 deg worst-case phase
margin -> new C205 220 pF C0G GUARD-GND (56 deg). Others pass.
simulations/system: chain matches SPICE (45.8 nV/rtHz at SR1), ADC
transparent, 21 mV rms 50 Hz clip level; J202 = 100 G recommended with
an insulated antenna (10 G if bare).
bom/: priced BOM ~516 EUR ex VAT, ~406 EUR with the recommended
cost-down set; details and part checks in bom/README.md. Both
transformers are now S22083 (S22082 not stocked anywhere).
Layout: GND fan-out before routing, hand-routed guard drive, DIP
supply buses, NPTH pour keep-outs.

Co-Authored-By: Claude Opus 5.5 <noreply@anthropic.com>
Claude-Session: https://claude.ai/code/session_01RsM1DhHhY1tSr2aHjVygSC
Parts:
- TR402: value S22082 -> S22083; MPN S22082 -> S22083
Changed lines of the file:
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@@
 		(on_board yes)
 		(dnp no)
-		(property "Reference" "#PWR091"
+		(property "Reference" "#PWR092"
 			(at 38.1 33.02 0)
 			(effects
@@
 			(project "antenna_amplifier"
 				(path "/61336681-2262-5f00-9d69-45832dcbe407/0ae99a2d-b679-543a-8f49-e431d07ea905"
-					(reference "#PWR091")
+					(reference "#PWR092")
 					(unit 1)
 				)
@@
 		(on_board yes)
 		(dnp no)
-		(property "Reference" "#PWR092"
+		(property "Reference" "#PWR093"
 			(at 38.1 58.42 0)
 			(effects
@@
 			(project "antenna_amplifier"
 				(path "/61336681-2262-5f00-9d69-45832dcbe407/0ae99a2d-b679-543a-8f49-e431d07ea905"
-					(reference "#PWR092")
+					(reference "#PWR093")
 					(unit 1)
 				)
@@
 		(on_board yes)
 		(dnp no)
-		(property "Reference" "#PWR093"
+		(property "Reference" "#PWR094"
 			(at 100.33 55.88 0)
 			(effects
@@
 			(project "antenna_amplifier"
 				(path "/61336681-2262-5f00-9d69-45832dcbe407/0ae99a2d-b679-543a-8f49-e431d07ea905"
-					(reference "#PWR093")
+					(reference "#PWR094")
 					(unit 1)
 				)
@@
 		(on_board yes)
 		(dnp no)
-		(property "Reference" "#PWR094"
+		(property "Reference" "#PWR095"
 			(at 100.33 68.58 0)
 			(effects
@@
 			(project "antenna_amplifier"
 				(path "/61336681-2262-5f00-9d69-45832dcbe407/0ae99a2d-b679-543a-8f49-e431d07ea905"
-					(reference "#PWR094")
+					(reference "#PWR095")
 					(unit 1)
 				)
@@
 		(on_board yes)
 		(dnp no)
-		(property "Reference" "#PWR095"
+		(property "Reference" "#PWR096"
 			(at 162.56 53.34 0)
 			(effects
@@
 			(project "antenna_amplifier"
 				(path "/61336681-2262-5f00-9d69-45832dcbe407/0ae99a2d-b679-543a-8f49-e431d07ea905"
-					(reference "#PWR095")
+					(reference "#PWR096")
 					(unit 1)
 				)
@@
 		(on_board yes)
 		(dnp no)
-		(property "Reference" "#PWR096"
+		(property "Reference" "#PWR097"
 			(at 203.2 86.36 0)
 			(effects
@@
 			(project "antenna_amplifier"
 				(path "/61336681-2262-5f00-9d69-45832dcbe407/0ae99a2d-b679-543a-8f49-e431d07ea905"
-					(reference "#PWR096")
+					(reference "#PWR097")
 					(unit 1)
 				)
@@
 		(on_board yes)
 		(dnp no)
-		(property "Reference" "#PWR097"
+		(property "Reference" "#PWR098"
 			(at 180.34 40.64 0)
 			(effects
@@
 			(project "antenna_amplifier"
 				(path "/61336681-2262-5f00-9d69-45832dcbe407/0ae99a2d-b679-543a-8f49-e431d07ea905"
-					(reference "#PWR097")
+					(reference "#PWR098")
 					(unit 1)
 				)
@@
 		(on_board yes)
 		(dnp no)
-		(property "Reference" "#PWR098"
+		(property "Reference" "#PWR099"
 			(at 182.88 96.52 0)
 			(effects
@@
 			(project "antenna_amplifier"
 				(path "/61336681-2262-5f00-9d69-45832dcbe407/0ae99a2d-b679-543a-8f49-e431d07ea905"
-					(reference "#PWR098")
+					(reference "#PWR099")
 					(unit 1)
 				)
@@
 		(on_board yes)
 		(dnp no)
-		(property "Reference" "#PWR099"
+		(property "Reference" "#PWR100"
 			(at 185.42 40.64 0)
 			(effects
@@
 			(project "antenna_amplifier"
 				(path "/61336681-2262-5f00-9d69-45832dcbe407/0ae99a2d-b679-543a-8f49-e431d07ea905"
-					(reference "#PWR099")
+					(reference "#PWR100")
 					(unit 1)
 				)
@@
 		(on_board yes)
 		(dnp no)
-		(property "Reference" "#PWR100"
+		(property "Reference" "#PWR101"
 			(at 124.46 118.11 0)
 			(effects
@@
 			(project "antenna_amplifier"
 				(path "/61336681-2262-5f00-9d69-45832dcbe407/0ae99a2d-b679-543a-8f49-e431d07ea905"
-					(reference "#PWR100")
+					(reference "#PWR101")
 					(unit 1)
 				)
@@
 		(on_board yes)
 		(dnp no)
-		(property "Reference" "#PWR101"
+		(property "Reference" "#PWR102"
 			(at 207.01 105.41 0)
 			(effects
@@
 			(project "antenna_amplifier"
 				(path "/61336681-2262-5f00-9d69-45832dcbe407/0ae99a2d-b679-543a-8f49-e431d07ea905"
-					(reference "#PWR101")
+					(reference "#PWR102")
 					(unit 1)
 				)
@@
 		(on_board yes)
 		(dnp no)
-		(property "Reference" "#PWR102"
+		(property "Reference" "#PWR103"
 			(at 207.01 118.11 0)
 			(effects
@@
 			(project "antenna_amplifier"
 				(path "/61336681-2262-5f00-9d69-45832dcbe407/0ae99a2d-b679-543a-8f49-e431d07ea905"
-					(reference "#PWR102")
+					(reference "#PWR103")
 					(unit 1)
 				)
@@
 		(on_board yes)
 		(dnp no)
-		(property "Reference" "#PWR103"
+		(property "Reference" "#PWR104"
 			(at 219.71 105.41 0)
 			(effects
@@
 			(project "antenna_amplifier"
 				(path "/61336681-2262-5f00-9d69-45832dcbe407/0ae99a2d-b679-543a-8f49-e431d07ea905"
-					(reference "#PWR103")
+					(reference "#PWR104")
 					(unit 1)
 				)
@@
 		(on_board yes)
 		(dnp no)
-		(property "Reference" "#PWR104"
+		(property "Reference" "#PWR105"
 			(at 219.71 118.11 0)
 			(effects
@@
 			(project "antenna_amplifier"
 				(path "/61336681-2262-5f00-9d69-45832dcbe407/0ae99a2d-b679-543a-8f49-e431d07ea905"
-					(reference "#PWR104")
+					(reference "#PWR105")
 					(unit 1)
 				)
@@
 		(on_board yes)
 		(dnp no)
-		(property "Reference" "#PWR105"
+		(property "Reference" "#PWR106"
 			(at 232.41 105.41 0)
 			(effects
@@
 			(project "antenna_amplifier"
 				(path "/61336681-2262-5f00-9d69-45832dcbe407/0ae99a2d-b679-543a-8f49-e431d07ea905"
-					(reference "#PWR105")
+					(reference "#PWR106")
 					(unit 1)
 				)
@@
 		(on_board yes)
 		(dnp no)
-		(property "Reference" "#PWR106"
+		(property "Reference" "#PWR107"
 			(at 232.41 118.11 0)
 			(effects
@@
 			(project "antenna_amplifier"
 				(path "/61336681-2262-5f00-9d69-45832dcbe407/0ae99a2d-b679-543a-8f49-e431d07ea905"
-					(reference "#PWR106")
+					(reference "#PWR107")
 					(unit 1)
 				)
@@
 		(on_board yes)
 		(dnp no)
-		(property "Reference" "#PWR107"
+		(property "Reference" "#PWR108"
 			(at 265.43 35.56 0)
 			(effects
@@
 			(project "antenna_amplifier"
 				(path "/61336681-2262-5f00-9d69-45832dcbe407/0ae99a2d-b679-543a-8f49-e431d07ea905"
-					(reference "#PWR107")
+					(reference "#PWR108")
 					(unit 1)
 				)
@@
 		(on_board yes)
 		(dnp no)
-		(property "Reference" "#PWR108"
+		(property "Reference" "#PWR109"
 			(at 308.61 57.15 0)
 			(effects
@@
 			(project "antenna_amplifier"
 				(path "/61336681-2262-5f00-9d69-45832dcbe407/0ae99a2d-b679-543a-8f49-e431d07ea905"
-					(reference "#PWR108")
+					(reference "#PWR109")
 					(unit 1)
 				)
@@
 		(on_board yes)
 		(dnp no)
-		(property "Reference" "#PWR109"
+		(property "Reference" "#PWR110"
 			(at 320.04 57.15 0)
 			(effects
@@
 			(project "antenna_amplifier"
 				(path "/61336681-2262-5f00-9d69-45832dcbe407/0ae99a2d-b679-543a-8f49-e431d07ea905"
-					(reference "#PWR109")
+					(reference "#PWR110")
 					(unit 1)
 				)
@@
 		(on_board yes)
 		(dnp no)
-		(property "Reference" "#PWR110"
+		(property "Reference" "#PWR111"
 			(at 331.47 57.15 0)
 			(effects
@@
 			(project "antenna_amplifier"
 				(path "/61336681-2262-5f00-9d69-45832dcbe407/0ae99a2d-b679-543a-8f49-e431d07ea905"
-					(reference "#PWR110")
+					(reference "#PWR111")
 					(unit 1)
 				)
@@
 		(on_board yes)
 		(dnp no)
-		(property "Reference" "#PWR111"
+		(property "Reference" "#PWR112"
 			(at 342.9 57.15 0)
 			(effects
@@
 			(project "antenna_amplifier"
 				(path "/61336681-2262-5f00-9d69-45832dcbe407/0ae99a2d-b679-543a-8f49-e431d07ea905"
-					(reference "#PWR111")
+					(reference "#PWR112")
 					(unit 1)
 				)
@@
 		(on_board yes)
 		(dnp no)
-		(property "Reference" "#PWR112"
+		(property "Reference" "#PWR113"
 			(at 354.33 57.15 0)
 			(effects
@@
 			(project "antenna_amplifier"
 				(path "/61336681-2262-5f00-9d69-45832dcbe407/0ae99a2d-b679-543a-8f49-e431d07ea905"
-					(reference "#PWR112")
+					(reference "#PWR113")
 					(unit 1)
 				)
@@
 		(on_board yes)
 		(dnp no)
-		(property "Reference" "#PWR113"
+		(property "Reference" "#PWR114"
 			(at 365.76 57.15 0)
 			(effects
@@
 			(project "antenna_amplifier"
 				(path "/61336681-2262-5f00-9d69-45832dcbe407/0ae99a2d-b679-543a-8f49-e431d07ea905"
-					(reference "#PWR113")
+					(reference "#PWR114")
 					(unit 1)
 				)
@@
 		(on_board yes)
 		(dnp no)
-		(property "Reference" "#PWR114"
+		(property "Reference" "#PWR115"
 			(at 377.19 57.15 0)
 			(effects
@@
 			(project "antenna_amplifier"
 				(path "/61336681-2262-5f00-9d69-45832dcbe407/0ae99a2d-b679-543a-8f49-e431d07ea905"
-					(reference "#PWR114")
+					(reference "#PWR115")
 					(unit 1)
 				)
@@
 		(on_board yes)
 		(dnp no)
-		(property "Reference" "#PWR115"
+		(property "Reference" "#PWR116"
 			(at 388.62 57.15 0)
 			(effects
@@
 			(project "antenna_amplifier"
 				(path "/61336681-2262-5f00-9d69-45832dcbe407/0ae99a2d-b679-543a-8f49-e431d07ea905"
-					(reference "#PWR115")
+					(reference "#PWR116")
 					(unit 1)
 				)
@@
 		(on_board yes)
 		(dnp no)
-		(property "Reference" "#PWR116"
+		(property "Reference" "#PWR117"
 			(at 152.4 179.07 0)
 			(effects
@@
 			(project "antenna_amplifier"
 				(path "/61336681-2262-5f00-9d69-45832dcbe407/0ae99a2d-b679-543a-8f49-e431d07ea905"
-					(reference "#PWR116")
+					(reference "#PWR117")
 					(unit 1)
 				)
@@
 		(on_board yes)
 		(dnp no)
-		(property "Reference" "#PWR117"
+		(property "Reference" "#PWR118"
 			(at 165.1 179.07 0)
 			(effects
@@
 			(project "antenna_amplifier"
 				(path "/61336681-2262-5f00-9d69-45832dcbe407/0ae99a2d-b679-543a-8f49-e431d07ea905"
-					(reference "#PWR117")
+					(reference "#PWR118")
 					(unit 1)
 				)
@@
 			)
 		)
-		(property "Value" "S22082"
+		(property "Value" "S22083"
 			(at 294.64 154.62 0)
 			(effects
@@
 			)
 		)
-		(property "MPN" "S22082"
+		(property "MPN" "S22083"
 			(at 302.26 160.02 0)
 			(effects
