File: PCB/antenna_amplifier/digital.kicad_sch (KiCad schematic)
At the start: 31 parts, among them J401 AES3 OUT, J402 S/PDIF OUT, SW401 CS8406 MODE, U401 CS8406, Y401 24.576MHz

Commit message: Leaded SOT23-5 oscillator (SiT2001B, Y402) fitted; SiT1602 kept as do-not-fit alternative
Hand-soldering friendly: Y402 sits under Y401 between the two clock series
resistors, both wired to OSC_OUT (outputs typed tri-state; fit only one).
Board re-routed: 0 DRC errors, 0 unconnected. Fitted parts get silkscreen
label priority over do-not-fit ones. Fab outputs now include populated STEP
models of both boards; BOM, assembly guide and open checks updated.

Co-Authored-By: Claude Opus 5.5 <noreply@anthropic.com>
Claude-Session: https://claude.ai/code/session_01RsM1DhHhY1tSr2aHjVygSC
Parts:
- added C408: 100n, Capacitor_SMD:C_0603_1608Metric, symbol Device:C
- added Y402: 24.576MHz, Package_TO_SOT_SMD:SOT-23-5, symbol antenna_amplifier:MEMS_OSC_SOT23
- Y401: now not fitted; now left out of the parts list
Connections:
- net +3V3: now also C408.1, Y402.3 (OE), Y402.4 (VDD)
- net GND: now also C408.2, Y402.1 (GND)
- net OSC_OUT: now also Y402.5 (OUT)
- no-connect marks 0 -> 1
Other:
- note added: "Fit Y402 (SOT23-5, leaded) or Y401 (3.2x2.5 no-lead), never both."

Commit message: Pedantic DRC/ERC pass: schematic parity clean, BNC notch, island without silk
- Board nets carry the schematic's names (sheet-path prefix on local nets, KiCad's
  unconnected-(...) nets on open pins): DRC schematic parity 0 on both boards.
- BNC: its mounting lugs reached 1.4 mm under the right-hand wall, whose round
  barrel hole left the bar resting on them (tilted wall, BNC shell = S/PDIF return
  shorted to the shield). The frame now has a 16 x 14 mm notch there, and the
  strip copper stops clear of the lugs. Micro-Fit notch widened to 14 mm.
- Guard island: mask opening follows the island outline; LMP7721 and the bias link
  use project footprint variants without silk on the island (no ink on the
  femtoamp surface). tools/fp_variants.py derives them from the stock footprints.
- S22083 footprint: silk outline no longer crosses its own slotted pads.
- CS8406 as a project symbol with pin 1 typed as the hardware-mode COPY/C input:
  ERC 0 on both schematics. PSU mounting holes out of the BOM; plate and PSU
  projects register the elara footprint library.
- Remaining amplifier DRC items: 79 solder-mask-bridge warnings, all on the
  deliberately unmasked guard island. PSU and plate boards: 0 of anything.

Co-Authored-By: Claude Opus 5.5 <noreply@anthropic.com>
Claude-Session: https://claude.ai/code/session_01RsM1DhHhY1tSr2aHjVygSC
Parts:
- U401: symbol Audio:CS8406 -> antenna_amplifier:CS8406_HW
Changed lines of the file:
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@@
 	)
 	(symbol
-		(lib_id "Audio:CS8406")
+		(lib_id "antenna_amplifier:CS8406_HW")
 		(at 182.88 68.58 0)
 		(unit 1)

Commit message: Pedantic schematic and silkscreen pass: zero overlaps, labels clear of tracks
Schematics
- tools/kicadgen/schcheck.py checks KiCad's own SVG rendering (exact stroke boxes)
  for text over text, lines through text, crowded twin labels and text outside the
  frame. Both schematics: 0 findings; ERC 0 on both.
- Generator: Sheet.join (one wire + one label instead of two facing labels),
  per-symbol field positions, per-pin stub lengths, shared power symbol for
  adjacent top/bottom rail pins, crowded rail runs get one label, longer PCM1804
  pins (no-connect cross clear of the pin number), PE value clear of its symbol.
- Fixed: doubled VIN_RAW/BIAS_DIV/LED_OVF/CV_ADJ/LED_C labels, +5VA vs VREG,
  +5V_PRE twins, CS8406 GND straps vs neighbours, BNC/LED/diode fields over their
  graphics, bucket-cell values vs tap labels, notes outside the frame, J2 -> J202.
- Root sheet: sub-sheets in signal-flow order with arrows and a design summary;
  dated title blocks.

Boards
- References prefer spots clear of tracks as well as parts (two candidate rings);
  compartment labels are re-placed after routing; the title block on the back is
  placed as one unit; no stitching via under any board text.
- DRC with schematic parity: amplifier 0 errors / 0 unconnected / 0 parity (only
  the intended bare-island mask warnings); PSU and plate 0 of anything.

Co-Authored-By: Claude Opus 5.5 <noreply@anthropic.com>
Claude-Session: https://claude.ai/code/session_01RsM1DhHhY1tSr2aHjVygSC
Other:
- moved on the sheet: J402

Commit message: Amplifier: single BNC, pluggable AES3, real 63 V Cg, wall clearances
From the placement and parts audit:
- J402 was an Amphenol 031-6575, a dual stacked BNC 29 mm tall that
  could never pass the 14 mm wall notch. Now a single right-angle
  B6252HB-NPP3G-50 (KiCad model), body inside the compartment and
  only the nut/barrel through the notch.
- J401's screw terminals sat under the right wall (screws at x = 194,
  wall from 193) and the shield mounts lid-down, so the AES3 cable could
  not be wired in place. Now a Phoenix MC 1,5/3-G-3,81 right-angle
  header: the MC 1,5/3-ST-3,81 plug is wired outside and pushed in
  through the notch (16 x 13 mm).
- C202's order code was the 100 VDC WIMA (24 x 45.5 mm) on a 35 mm
  footprint. Now MKS4C061007G00KSSD (63 VDC, 41.5 x 20 x 39.5 mm) on the
  matching footprint; C301 on its real 8.5 mm footprint.
- J101 moved 1.5 mm so its body is centred in its notch (was 0.6 mm
  from the notch side); C101, C205 and TR402 moved off the walls.
- ANT_BIAS leaves the island stub through a via so it can reach In2.
- Fab-layer values hidden on both boards: the assembly drawing now shows
  clean references (values are in the BOMs). The STEP export uses the
  board corner as origin for the mechanical fit checks.
DRC: amplifier 77 intended island mask bridges only, PSU 0; unconnected
0 and parity 0 on both; ERC 0; schematic legibility 0.

Co-Authored-By: Claude Opus 5.5 <noreply@anthropic.com>
Claude-Session: https://claude.ai/code/session_01RsM1DhHhY1tSr2aHjVygSC
Parts:
- J401: footprint TerminalBlock_Phoenix:TerminalBlock_Phoenix_MKDS-1,5-3-5.08_1x03_P5.08mm_Horizontal -> Connector_Phoenix_MC:PhoenixContact_MC_1,5_3-G-3.81_1x03_P3.81mm_Horizontal; MPN 1715734 -> 1803280 + 1803581 plug
- J402: footprint Connector_Coaxial:BNC_Amphenol_031-6575_Horizontal -> Connector_Coaxial:BNC_Amphenol_B6252HB-NPP3G-50_Horizontal; MPN 031-6575 -> B6252HB-NPP3G-50; Manufacturer Amphenol RF -> Amphenol
Changed lines of the file:
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@@
 			)
 		)
-		(property "Footprint" "TerminalBlock_Phoenix:TerminalBlock_Phoenix_MKDS-1,5-3-5.08_1x03_P5.08mm_Horizontal"
+		(property "Footprint" "Connector_Phoenix_MC:PhoenixContact_MC_1,5_3-G-3.81_1x03_P3.81mm_Horizontal"
 			(at 129.54 160.02 0)
 			(effects
@@
 			)
 		)
-		(property "Description" "AES3 cable: 1 shield (open by default), 2 hot, 3 cold"
+		(property "Description" "AES3 cable, pluggable through the wall notch: MC 1,5/3-G-3,81 header + MC 1,5/3-ST-3,81 plug; 1 shield (open by default), 2 hot, 3 cold"
 			(at 129.54 160.02 0)
 			(effects
@@
 			)
 		)
-		(property "MPN" "1715734"
+		(property "MPN" "1803280 + 1803581 plug"
 			(at 129.54 160.02 0)
 			(effects
@@
 			)
 		)
-		(property "Footprint" "Connector_Coaxial:BNC_Amphenol_031-6575_Horizontal"
+		(property "Footprint" "Connector_Coaxial:BNC_Amphenol_B6252HB-NPP3G-50_Horizontal"
 			(at 347.98 160.02 0)
 			(effects
@@
 			)
 		)
-		(property "Description" "BNC right-angle PCB jack, S/PDIF coax (BNC-RCA adapter)"
+		(property "Description" "BNC right-angle PCB jack (single); shell = S/PDIF return, transformer-isolated from GND, so it must not touch the shield wall"
 			(at 347.98 160.02 0)
 			(effects
@@
 			)
 		)
-		(property "Manufacturer" "Amphenol RF"
+		(property "Manufacturer" "Amphenol"
 			(at 347.98 160.02 0)
 			(effects
@@
 			)
 		)
-		(property "MPN" "031-6575"
+		(property "MPN" "B6252HB-NPP3G-50"
 			(at 347.98 160.02 0)
 			(effects

Commit message: Battery-friendly amplifier, RJ45 AES3 output, tidy placement, 1 mm PSU barrier
Amplifier schematic:
- No LEDs (battery use): the D301 overflow LED becomes test point TP301.
- PCM1804 FMT/S-M/OSR pins use the chip's internal 51 k pull-downs (6 resistors
  gone); BYPAS and the CS8406 mode pins get 47 k: about 3 mA less on +3V3.
- One output: AES3 on a shielded RJ45 (Amphenol RJHSE-5380, blue pair 4/5) for
  shielded twisted-pair cable, transformer isolated; the cable shield floats at
  the receiver (10 nF RF bond DNP, the DC bond is gone). The S/PDIF coax branch
  (BNC, second S22083, 5.6 mA standing current) is removed.

Layout:
- Amplifier re-placed in functional blocks on a 0.5 mm grid: PCM1804 and CS8406
  side by side so the I2S lines run straight, capacitor cells round the LDOs,
  DIP pull-downs in line with the switch pins, guard column in signal order with
  a re-routed hand guard-drive link. RJ45 notch 20 x 16 mm, BNC notch gone.
- PSU tidied (aligned columns, flyback diodes over their relays) and the charger
  / receiver copper kept >= 1.0 mm apart (was 0.30 mm): custom DRC rule, 1 mm
  router class for the relay contacts, hand-routed GND / GND_C at the relays.
- Reference labels follow each part's row; every label on silk except on the
  bare guard island. Fixed two placer bugs: each label counted as its own
  obstacle (SWIG proxies compared with 'is'), and unplaced labels blocked their
  neighbours. Texts are measured by their strokes, not KiCad's text cell.

Mechanics: RJ45 notch, plug envelope and a 1 mm isolation gap in fit_check.
BOM: 502 EUR as designed, 407 EUR recommended; 81 order lines.
Docs: STATUS, PLAN, ASSEMBLY, MOUNTING, README, mechanical and BOM notes;
MAINS_CABLE gains a certified DIY screened-cable option (H07RN-F + foil + braid)
and says why Ethernet cable must not carry mains.

All checks pass (tools/check_all.sh): ERC 0, DRC/parity 0 on all boards (only
the intended guard-island mask bridges), mains clearances, fit check, 27 tests.

Co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
Parts:
- removed C408: 100n, Capacitor_SMD:C_0603_1608Metric, symbol Device:C
- removed J402: S/PDIF OUT, Connector_Coaxial:BNC_Amphenol_B6252HB-NPP3G-50_Horizontal, symbol Connector:Conn_Coaxial
- removed R414: 0, Resistor_SMD:R_0603_1608Metric, symbol Device:R
- removed R415, R416: 249, Resistor_SMD:R_0603_1608Metric, symbol Device:R
- removed R417: 90.9, Resistor_SMD:R_0603_1608Metric, symbol Device:R
- removed TR402: S22083, elara:Transformer_Pulse_4Pin_W7.62mm, symbol antenna_amplifier:XFMR_1to1
- C406: Role optional RF bond -> optional RF bond of the cable shield (keeps the DC isolatio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
- C407: Role DC block -> (none)
- J401: footprint Connector_Phoenix_MC:PhoenixContact_MC_1,5_3-G-3.81_1x03_P3.81mm_Horizontal -> Connector_RJ:RJ45_Amphenol_RJHSE5380; symbol Connector:Screw_Terminal_01x03 -> Connector:RJ45_Shielded; MPN 1803280 + 1803581 plug -> RJHSE-5380; Manufacturer Phoenix Contact -> Amphenol
- R403, R404, R405, R406, R407, R408, R409, R410, R411: value 10k -> 47k; MPN ERA-3AEB103V -> ERA-3AEB473V
Connections:
- net COAX_A is gone; now on net +3V3: C407.1
- net COAX_P1 is gone; now on net GND: C407.2
- net AES_COLD: now also J401.5; no longer J401.3 (Pin_3)
- net AES_HOT: now also J401.4; no longer J401.2 (Pin_2)
- net AES_SHIELD: now also J401.SH; no longer J401.1 (Pin_1)
- no-connect marks 1 -> 7
Other:
- note added: "AES3 OUTPUT transformer isolated, RJ45 for shielded twisted pair"
- note added: "Cable: shielded Cat5e/6 (100 R pairs), shield connected at the indoor end only. AES3 is polarity-free."
- note removed: "OUTPUTS transformer isolated"
- note removed: "S/PDIF 75 R coax, 0.5 Vpp"
- note removed: "S/PDIF: 2 x 249 R + 90.9 R shunt: 75 R source, 0.5 Vpp into 75 R."
- title: ELARA antenna amplifier - Clock and S/PDIF + AES3 output -> ELARA antenna amplifier - Clock and AES3 output
- moved on the sheet: C406, C407
