File: PCB/antenna_amplifier/frontend.kicad_sch (KiCad schematic)
At the start: 22 parts, among them J201 FILT_IN, J202 BIAS, U201 LMP7721, U202 LMP7715, U203 LMP7715

Commit message: Apply simulation fixes; add PSU/stability/system sims and priced BOM
simulations/psu: the charger caps each bucket at ~10.3 V, so the LT3045
at 8.45 V dropped out. Now R_SET 69.8k (6.98 V) and a 15 s swap
(CD4060 Rt 80.6k): +1.97 V headroom nominal, +0.49 V worst corner.
Charger output cap 10 uF -> 100 nF (3 A cold-start contact spike).
Swap artefact >= 83 dB below the floor; 50 Hz leakage 4-5 orders lower
than a direct AC-DC module (earth the receiver ground locally).
simulations/stability: guard buffer U202 had 43 deg worst-case phase
margin -> new C205 220 pF C0G GUARD-GND (56 deg). Others pass.
simulations/system: chain matches SPICE (45.8 nV/rtHz at SR1), ADC
transparent, 21 mV rms 50 Hz clip level; J202 = 100 G recommended with
an insulated antenna (10 G if bare).
bom/: priced BOM ~516 EUR ex VAT, ~406 EUR with the recommended
cost-down set; details and part checks in bom/README.md. Both
transformers are now S22083 (S22082 not stocked anywhere).
Layout: GND fan-out before routing, hand-routed guard drive, DIP
supply buses, NPTH pour keep-outs.

Co-Authored-By: Claude Opus 5.5 <noreply@anthropic.com>
Claude-Session: https://claude.ai/code/session_01RsM1DhHhY1tSr2aHjVygSC
Parts:
- added C208: 100n, Capacitor_SMD:C_0603_1608Metric, symbol Device:C
- C205: value 100n -> 220p; MPN GRM188R71H104KA93D -> GRM1885C1H221JA01D; Role (none) -> guard buffer stability (PM 43 -> 56 deg)
- C206: value 4700u -> 100n; footprint Capacitor_THT:CP_Radial_D16.0mm_P7.50mm -> Capacitor_SMD:C_0603_1608Metric; symbol Device:C_Polarized -> Device:C; MPN EEU-FR1C472 -> GRM188R71H104KA93D; Manufacturer Panasonic -> Murata; Role divider noise filter, 1.4 mHz -> (none)
- C207: value 100n -> 4700u; footprint Capacitor_SMD:C_0603_1608Metric -> Capacitor_THT:CP_Radial_D16.0mm_P7.50mm; symbol Device:C -> Device:C_Polarized; MPN GRM188R71H104KA93D -> EEU-FR1C472; Manufacturer Murata -> Panasonic; Role (none) -> divider noise filter, 1.4 mHz
Connections:
- net +5V_PRE: now also C206.1, C208.1; no longer C205.1, C207.1
- net BIAS_DIV: now also C207.1; no longer C206.1
- net GND: now also C208.2
- net GUARD: now also C205.1
Other:
- moved on the sheet: C205
Changed lines of the file:
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@@
+	(symbol
+		(lib_id "Device:C")
+		(at 262.89 55.88 0)
+		(unit 1)
+		(exclude_from_sim no)
+		(in_bom yes)
+		(on_board yes)
+		(dnp no)
+		(property "Reference" "C205"
+			(at 265.72 54.88 0)
+			(effects
+				(font
+					(size 1.27 1.27)
+				)
+				(justify left)
+			)
+		)
+		(property "Value" "220p"
+			(at 265.72 57.48 0)
+			(effects
+				(font
+					(size 1.27 1.27)
+				)
+				(justify left)
+			)
+		)
+		(property "Footprint" "Capacitor_SMD:C_0603_1608Metric"
+			(at 262.89 55.88 0)
+			(effects
+				(font
+					(size 1.27 1.27)
+				)
+				(hide yes)
+			)
+		)
+		(property "Datasheet" "~"
+			(at 262.89 55.88 0)
+			(effects
+				(font
+					(size 1.27 1.27)
+				)
+				(hide yes)
+			)
+		)
+		(property "Description" "MLCC 220p 50V C0G 0603 (guard stability)"
+			(at 262.89 55.88 0)
+			(effects
+				(font
+					(size 1.27 1.27)
+				)
+				(hide yes)
+			)
+		)
+		(property "Manufacturer" "Murata"
+			(at 262.89 55.88 0)
+			(effects
+				(font
+					(size 1.27 1.27)
+				)
+				(hide yes)
+			)
+		)
+		(property "MPN" "GRM1885C1H221JA01D"
+			(at 262.89 55.88 0)
+			(effects
+				(font
+					(size 1.27 1.27)
+				)
+				(hide yes)
+			)
+		)
+		(property "Role" "guard buffer stability (PM 43 -> 56 deg)"
+			(at 262.89 55.88 0)
+			(effects
+				(font
+					(size 1.27 1.27)
+				)
+				(hide yes)
+			)
+		)
+		(pin "1"
+		)
+		(pin "2"
+		)
+		(instances
+			(project "antenna_amplifier"
+				(path "/61336681-2262-5f00-9d69-45832dcbe407/90e2f3c2-8af3-5a43-a380-6e41c0a9f4da"
+					(reference "C205")
+					(unit 1)
+				)
+			)
+		)
+	)
+	(wire
+		(pts (xy 262.89 52.07) (xy 262.89 49.53))
+		(stroke
+			(width 0)
+			(type default)
+		)
+	)
+	(label "GUARD"
+		(at 262.89 49.53 90)
+		(fields_autoplaced yes)
+		(effects
+			(font
+				(size 1.27 1.27)
+			)
+			(justify left bottom)
+		)
+	)
+	(wire
+		(pts (xy 262.89 59.69) (xy 262.89 62.23))
+		(stroke
+			(width 0)
+			(type default)
+		)
+	)
+	(symbol
+		(lib_id "power:GND")
+		(at 262.89 62.23 0)
+		(unit 1)
+		(exclude_from_sim no)
+		(in_bom yes)
+		(on_board yes)
+		(dnp no)
+		(property "Reference" "#PWR043"
+			(at 262.89 62.23 0)
+			(effects
+				(font
+					(size 1.27 1.27)
+				)
+				(hide yes)
+			)
+		)
+		(property "Value" "GND"
+			(at 262.89 66.53 0)
+			(effects
+				(font
+					(size 1.27 1.27)
+				)
+			)
+		)
+		(property "Footprint" ""
+			(at 262.89 62.23 0)
+			(effects
+				(font
+					(size 1.27 1.27)
+				)
+				(hide yes)
+			)
+		)
+		(property "Datasheet" ""
+			(at 262.89 62.23 0)
+			(effects
+				(font
+					(size 1.27 1.27)
+				)
+				(hide yes)
+			)
+		)
+		(property "Description" ""
+			(at 262.89 62.23 0)
+			(effects
+				(font
+					(size 1.27 1.27)
+				)
+				(hide yes)
+			)
+		)
+		(pin "1"
+		)
+		(instances
+			(project "antenna_amplifier"
+				(path "/61336681-2262-5f00-9d69-45832dcbe407/90e2f3c2-8af3-5a43-a380-6e41c0a9f4da"
+					(reference "#PWR043")
+					(unit 1)
+				)
+			)
+		)
+	)
 	(symbol
 		(lib_id "Device:C")
@@
 		(on_board yes)
 		(dnp no)
-		(property "Reference" "C205"
+		(property "Reference" "C206"
 			(at 274.61 49.8 0)
 			(effects
@@
 			(project "antenna_amplifier"
 				(path "/61336681-2262-5f00-9d69-45832dcbe407/90e2f3c2-8af3-5a43-a380-6e41c0a9f4da"
-					(reference "C205")
+					(reference "C206")
 					(unit 1)
 				)
@@
 		(on_board yes)
 		(dnp no)
-		(property "Reference" "#PWR043"
+		(property "Reference" "#PWR044"
 			(at 271.78 44.45 0)
 			(effects
@@
 			(project "antenna_amplifier"
 				(path "/61336681-2262-5f00-9d69-45832dcbe407/90e2f3c2-8af3-5a43-a380-6e41c0a9f4da"
-					(reference "#PWR043")
+					(reference "#PWR044")
 					(unit 1)
 				)
@@
 		(on_board yes)
 		(dnp no)
-		(property "Reference" "#PWR044"
+		(property "Reference" "#PWR045"
 			(at 271.78 57.15 0)
 			(effects
@@
 			(project "antenna_amplifier"
 				(path "/61336681-2262-5f00-9d69-45832dcbe407/90e2f3c2-8af3-5a43-a380-6e41c0a9f4da"
-					(reference "#PWR044")
+					(reference "#PWR045")
 					(unit 1)
 				)
@@
 		(on_board yes)
 		(dnp no)
-		(property "Reference" "#PWR045"
+		(property "Reference" "#PWR046"
 			(at 27.94 111.76 0)
 			(effects
@@
 			(project "antenna_amplifier"
 				(path "/61336681-2262-5f00-9d69-45832dcbe407/90e2f3c2-8af3-5a43-a380-6e41c0a9f4da"
-					(reference "#PWR045")
+					(reference "#PWR046")
 					(unit 1)
 				)
@@
 		(on_board yes)
 		(dnp no)
-		(property "Reference" "#PWR046"
+		(property "Reference" "#PWR047"
 			(at 27.94 153.67 0)
 			(effects
@@
 			(project "antenna_amplifier"
 				(path "/61336681-2262-5f00-9d69-45832dcbe407/90e2f3c2-8af3-5a43-a380-6e41c0a9f4da"
-					(reference "#PWR046")
+					(reference "#PWR047")
 					(unit 1)
 				)
@@
 		(on_board yes)
 		(dnp no)
-		(property "Reference" "C206"
+		(property "Reference" "C207"
 			(at 43.73 143.78 0)
 			(effects
@@
 			(project "antenna_amplifier"
 				(path "/61336681-2262-5f00-9d69-45832dcbe407/90e2f3c2-8af3-5a43-a380-6e41c0a9f4da"
-					(reference "C206")
+					(reference "C207")
 					(unit 1)
 				)
@@
 		(on_board yes)
 		(dnp no)
-		(property "Reference" "#PWR047"
+		(property "Reference" "#PWR048"
 			(at 40.64 151.13 0)
 			(effects
@@
 			(project "antenna_amplifier"
 				(path "/61336681-2262-5f00-9d69-45832dcbe407/90e2f3c2-8af3-5a43-a380-6e41c0a9f4da"
-					(reference "#PWR047")
+					(reference "#PWR048")
 					(unit 1)
 				)
@@
 		(on_board yes)
 		(dnp no)
-		(property "Reference" "#PWR048"
+		(property "Reference" "#PWR049"
 			(at 80.01 116.84 0)
 			(effects
@@
 			(project "antenna_amplifier"
 				(path "/61336681-2262-5f00-9d69-45832dcbe407/90e2f3c2-8af3-5a43-a380-6e41c0a9f4da"
-					(reference "#PWR048")
+					(reference "#PWR049")
 					(unit 1)
 				)
@@
 		(on_board yes)
 		(dnp no)
-		(property "Reference" "#PWR049"
+		(property "Reference" "#PWR050"
 			(at 80.01 137.16 0)
 			(effects
@@
 			(project "antenna_amplifier"
 				(path "/61336681-2262-5f00-9d69-45832dcbe407/90e2f3c2-8af3-5a43-a380-6e41c0a9f4da"
-					(reference "#PWR049")
+					(reference "#PWR050")
 					(unit 1)
 				)
@@
 		(on_board yes)
 		(dnp no)
-		(property "Reference" "C207"
+		(property "Reference" "C208"
 			(at 169.2 143.78 0)
 			(effects
@@
 			(project "antenna_amplifier"
 				(path "/61336681-2262-5f00-9d69-45832dcbe407/90e2f3c2-8af3-5a43-a380-6e41c0a9f4da"
-					(reference "C207")
+					(reference "C208")
 					(unit 1)
 				)
@@
 		(on_board yes)
 		(dnp no)
-		(property "Reference" "#PWR050"
+		(property "Reference" "#PWR051"
 			(at 166.37 138.43 0)
 			(effects
@@
 			(project "antenna_amplifier"
 				(path "/61336681-2262-5f00-9d69-45832dcbe407/90e2f3c2-8af3-5a43-a380-6e41c0a9f4da"
-					(reference "#PWR050")
+					(reference "#PWR051")
 					(unit 1)
 				)
@@
 		(on_board yes)
 		(dnp no)
-		(property "Reference" "#PWR051"
+		(property "Reference" "#PWR052"
 			(at 166.37 151.13 0)
 			(effects
@@
 			(project "antenna_amplifier"
 				(path "/61336681-2262-5f00-9d69-45832dcbe407/90e2f3c2-8af3-5a43-a380-6e41c0a9f4da"
-					(reference "#PWR051")
+					(reference "#PWR052")
 					(unit 1)
 				)
@@
 		(on_board yes)
 		(dnp no)
-		(property "Reference" "#PWR052"
+		(property "Reference" "#PWR053"
 			(at 261.62 93.98 0)
 			(effects
@@
 			(project "antenna_amplifier"
 				(path "/61336681-2262-5f00-9d69-45832dcbe407/90e2f3c2-8af3-5a43-a380-6e41c0a9f4da"
-					(reference "#PWR052")
-					(unit 1)
-				)
+					(reference "#PWR053")
+					(unit 1)
+				)

Commit message: Pedantic DRC/ERC pass: schematic parity clean, BNC notch, island without silk
- Board nets carry the schematic's names (sheet-path prefix on local nets, KiCad's
  unconnected-(...) nets on open pins): DRC schematic parity 0 on both boards.
- BNC: its mounting lugs reached 1.4 mm under the right-hand wall, whose round
  barrel hole left the bar resting on them (tilted wall, BNC shell = S/PDIF return
  shorted to the shield). The frame now has a 16 x 14 mm notch there, and the
  strip copper stops clear of the lugs. Micro-Fit notch widened to 14 mm.
- Guard island: mask opening follows the island outline; LMP7721 and the bias link
  use project footprint variants without silk on the island (no ink on the
  femtoamp surface). tools/fp_variants.py derives them from the stock footprints.
- S22083 footprint: silk outline no longer crosses its own slotted pads.
- CS8406 as a project symbol with pin 1 typed as the hardware-mode COPY/C input:
  ERC 0 on both schematics. PSU mounting holes out of the BOM; plate and PSU
  projects register the elara footprint library.
- Remaining amplifier DRC items: 79 solder-mask-bridge warnings, all on the
  deliberately unmasked guard island. PSU and plate boards: 0 of anything.

Co-Authored-By: Claude Opus 5.5 <noreply@anthropic.com>
Claude-Session: https://claude.ai/code/session_01RsM1DhHhY1tSr2aHjVygSC
Parts:
- J202: footprint Connector_PinHeader_2.54mm:PinHeader_1x02_P2.54mm_Vertical -> elara:PinHeader_1x02_P2.54mm_Vertical_NoSilk
- U201: footprint Package_SO:SOIC-8_3.9x4.9mm_P1.27mm -> elara:SOIC-8_3.9x4.9mm_P1.27mm_GuardIsland
Changed lines of the file:
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@@
 			)
 		)
-		(property "Footprint" "Connector_PinHeader_2.54mm:PinHeader_1x02_P2.54mm_Vertical"
+		(property "Footprint" "elara:PinHeader_1x02_P2.54mm_Vertical_NoSilk"
 			(at 27.94 55.88 0)
 			(effects
@@
 			)
 		)
-		(property "Footprint" "Package_SO:SOIC-8_3.9x4.9mm_P1.27mm"
+		(property "Footprint" "elara:SOIC-8_3.9x4.9mm_P1.27mm_GuardIsland"
 			(at 104.14 45.72 0)
 			(effects

Commit message: Pedantic schematic and silkscreen pass: zero overlaps, labels clear of tracks
Schematics
- tools/kicadgen/schcheck.py checks KiCad's own SVG rendering (exact stroke boxes)
  for text over text, lines through text, crowded twin labels and text outside the
  frame. Both schematics: 0 findings; ERC 0 on both.
- Generator: Sheet.join (one wire + one label instead of two facing labels),
  per-symbol field positions, per-pin stub lengths, shared power symbol for
  adjacent top/bottom rail pins, crowded rail runs get one label, longer PCM1804
  pins (no-connect cross clear of the pin number), PE value clear of its symbol.
- Fixed: doubled VIN_RAW/BIAS_DIV/LED_OVF/CV_ADJ/LED_C labels, +5VA vs VREG,
  +5V_PRE twins, CS8406 GND straps vs neighbours, BNC/LED/diode fields over their
  graphics, bucket-cell values vs tap labels, notes outside the frame, J2 -> J202.
- Root sheet: sub-sheets in signal-flow order with arrows and a design summary;
  dated title blocks.

Boards
- References prefer spots clear of tracks as well as parts (two candidate rings);
  compartment labels are re-placed after routing; the title block on the back is
  placed as one unit; no stitching via under any board text.
- DRC with schematic parity: amplifier 0 errors / 0 unconnected / 0 parity (only
  the intended bare-island mask warnings); PSU and plate 0 of anything.

Co-Authored-By: Claude Opus 5.5 <noreply@anthropic.com>
Claude-Session: https://claude.ai/code/session_01RsM1DhHhY1tSr2aHjVygSC
Other:
- note added: "J202: fit the G-ohm bias R."
- note removed: "J2: fit G-ohm bias R"
- moved on the sheet: U202

Commit message: Amplifier: single BNC, pluggable AES3, real 63 V Cg, wall clearances
From the placement and parts audit:
- J402 was an Amphenol 031-6575, a dual stacked BNC 29 mm tall that
  could never pass the 14 mm wall notch. Now a single right-angle
  B6252HB-NPP3G-50 (KiCad model), body inside the compartment and
  only the nut/barrel through the notch.
- J401's screw terminals sat under the right wall (screws at x = 194,
  wall from 193) and the shield mounts lid-down, so the AES3 cable could
  not be wired in place. Now a Phoenix MC 1,5/3-G-3,81 right-angle
  header: the MC 1,5/3-ST-3,81 plug is wired outside and pushed in
  through the notch (16 x 13 mm).
- C202's order code was the 100 VDC WIMA (24 x 45.5 mm) on a 35 mm
  footprint. Now MKS4C061007G00KSSD (63 VDC, 41.5 x 20 x 39.5 mm) on the
  matching footprint; C301 on its real 8.5 mm footprint.
- J101 moved 1.5 mm so its body is centred in its notch (was 0.6 mm
  from the notch side); C101, C205 and TR402 moved off the walls.
- ANT_BIAS leaves the island stub through a via so it can reach In2.
- Fab-layer values hidden on both boards: the assembly drawing now shows
  clean references (values are in the BOMs). The STEP export uses the
  board corner as origin for the mechanical fit checks.
DRC: amplifier 77 intended island mask bridges only, PSU 0; unconnected
0 and parity 0 on both; ERC 0; schematic legibility 0.

Co-Authored-By: Claude Opus 5.5 <noreply@anthropic.com>
Claude-Session: https://claude.ai/code/session_01RsM1DhHhY1tSr2aHjVygSC
Parts:
- C202: footprint Capacitor_THT:C_Rect_L41.5mm_W35.0mm_P37.50mm_MKS4 -> Capacitor_THT:C_Rect_L41.5mm_W20.0mm_P37.50mm_MKS4; MPN MKS4 100uF 63V PCM37.5 -> MKS4C061007G00KSSD
Changed lines of the file:
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@@
 			)
 		)
-		(property "Footprint" "Capacitor_THT:C_Rect_L41.5mm_W35.0mm_P37.50mm_MKS4"
+		(property "Footprint" "Capacitor_THT:C_Rect_L41.5mm_W20.0mm_P37.50mm_MKS4"
 			(at 97.79 78.74 0)
 			(effects
@@
 			)
 		)
-		(property "Description" "Film 100u 63V PET, PCM 37.5 mm (Cg)"
+		(property "Description" "Film 100u 63 VDC PET, PCM 37.5 mm, 41.5 x 20 x 39.5 mm (Cg)"
 			(at 97.79 78.74 0)
 			(effects
@@
 			)
 		)
-		(property "MPN" "MKS4 100uF 63V PCM37.5"
+		(property "MPN" "MKS4C061007G00KSSD"
 			(at 97.79 78.74 0)
 			(effects

Commit message: LMP7721 pinout corrected: inputs on pins 1/8, OUT on 4, V+ on 6, V- on 3
The project symbol had IN- on pin 3, GND on 4, OUT on 6 and V+ on 8; as
drawn, the board would have shorted the op-amp's output to GND. The
LMP7721 has both inputs at one end (1 = +IN, 8 = -IN), the N/C isolation
pins 2 and 7 (tied to the guard) next to them, V- on 3, OUT on 4 and V+
on 6 (TI datasheet and evaluation-board notes).

The guard ring already suited the real pinout (inputs at the pin 1/8 end,
guard bar under the body joining pins 2 and 7). Re-placed around U201:
Rf, Cf, Rg and the guard buffer in one column north-east of the chip on a
single hand-routed spine from pin 8; the guard drive (R203, C205) enters
the ring at its north-east corner; V+ decoupling beside pin 6; the V- via
under the body, with nothing else routed there, so OUT leaves pin 4
southwards on In2. HWCK1, which Freerouting now walls in, is pre-routed on
its previous path, and 'finish' removes the router's dangling stubs.
DRC/ERC/parity clean, every label on silk except the two on the bare
island, fit check OK.

Co-Authored-By: Claude Opus 5.5 <noreply@anthropic.com>
Claude-Session: https://claude.ai/code/session_01RsM1DhHhY1tSr2aHjVygSC
Connections:
- net +5V_PRE: now also U201.6; no longer U201.8
- net GND: now also U201.3; no longer U201.4
- net IN_N: now also U201.8 (-); no longer U201.3 (-)
- net PREAMP_OUT: now also U201.4; no longer U201.6
Changed lines of the file:
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@@
 			)
 		)
-		(property "Description" "Electrometer op-amp, 3 fA bias, guard pins 2/7"
+		(property "Description" "Electrometer op-amp, 3 fA, inputs pins 1/8, guard pins 2/7"
 			(at 104.14 45.72 0)
 			(effects
@@
 		(pin "1"
 		)
-		(pin "3"
-		)
-		(pin "6"
-		)
 		(pin "8"
 		)
 		(pin "4"
 		)
+		(pin "6"
+		)
+		(pin "3"
+		)
 		(pin "2"
