File: PCB/acdc_converter/acdc_converter.kicad_pcb (KiCad board)
At the start: 2 copper layers, 150 x 90 mm, 64 parts, among them J1 MAINS L N PE, J2 9V OUT, K1 G6K-2F-Y DC12, K2 G6K-2F-Y DC12, Q1 2N7002, U1 LM317, U2 LM317, U3 L78L12, U4 CD4060B, U5 LT3045

Commit message: Pedantic DRC/ERC pass: schematic parity clean, BNC notch, island without silk
- Board nets carry the schematic's names (sheet-path prefix on local nets, KiCad's
  unconnected-(...) nets on open pins): DRC schematic parity 0 on both boards.
- BNC: its mounting lugs reached 1.4 mm under the right-hand wall, whose round
  barrel hole left the bar resting on them (tilted wall, BNC shell = S/PDIF return
  shorted to the shield). The frame now has a 16 x 14 mm notch there, and the
  strip copper stops clear of the lugs. Micro-Fit notch widened to 14 mm.
- Guard island: mask opening follows the island outline; LMP7721 and the bias link
  use project footprint variants without silk on the island (no ink on the
  femtoamp surface). tools/fp_variants.py derives them from the stock footprints.
- S22083 footprint: silk outline no longer crosses its own slotted pads.
- CS8406 as a project symbol with pin 1 typed as the hardware-mode COPY/C input:
  ERC 0 on both schematics. PSU mounting holes out of the BOM; plate and PSU
  projects register the elara footprint library.
- Remaining amplifier DRC items: 79 solder-mask-bridge warnings, all on the
  deliberately unmasked guard island. PSU and plate boards: 0 of anything.

Co-Authored-By: Claude Opus 5.5 <noreply@anthropic.com>
Claude-Session: https://claude.ai/code/session_01RsM1DhHhY1tSr2aHjVygSC
Connections:
- net AC_L renamed /Two-bucket isolated supply/AC_L
- net AC_N renamed /Two-bucket isolated supply/AC_N
- net A_1 renamed /Two-bucket isolated supply/A_1
- net A_2 renamed /Two-bucket isolated supply/A_2
- net A_3 renamed /Two-bucket isolated supply/A_3
- net A_N renamed /Two-bucket isolated supply/A_N
- net A_P renamed /Two-bucket isolated supply/A_P
- net B_1 renamed /Two-bucket isolated supply/B_1
- net B_2 renamed /Two-bucket isolated supply/B_2
- net B_3 renamed /Two-bucket isolated supply/B_3
- net B_N renamed /Two-bucket isolated supply/B_N
- net B_P renamed /Two-bucket isolated supply/B_P
- net CC_OUT renamed /Two-bucket isolated supply/CC_OUT
- net CC_SET renamed /Two-bucket isolated supply/CC_SET
- net CHG renamed /Two-bucket isolated supply/CHG
- net CHG_A renamed /Two-bucket isolated supply/CHG_A
- net CHG_B renamed /Two-bucket isolated supply/CHG_B
- net CHG_D renamed /Two-bucket isolated supply/CHG_D
- net COIL_N renamed /Two-bucket isolated supply/COIL_N
- net CV_ADJ renamed /Two-bucket isolated supply/CV_ADJ
- net GATE renamed /Two-bucket isolated supply/GATE
- net LED_C renamed /Two-bucket isolated supply/LED_C
- net LOAD_A renamed /Two-bucket isolated supply/LOAD_A
- net LOAD_B renamed /Two-bucket isolated supply/LOAD_B
- net LOAD_P renamed /Two-bucket isolated supply/LOAD_P
- net L_IN renamed /Two-bucket isolated supply/L_IN
- net OSC_C renamed /Two-bucket isolated supply/OSC_C
- net OSC_I renamed /Two-bucket isolated supply/OSC_I
- net OSC_R renamed /Two-bucket isolated supply/OSC_R
- net OSC_X renamed /Two-bucket isolated supply/OSC_X
- net OUT_N renamed /Two-bucket isolated supply/OUT_N
- net SET renamed /Two-bucket isolated supply/SET
- net SWAP renamed /Two-bucket isolated supply/SWAP
- net VREG renamed /Two-bucket isolated supply/VREG
- U4 pad 1: (no net) -> unconnected-(U4-Q12-Pad1)
- U4 pad 13: (no net) -> unconnected-(U4-Q9-Pad13)
- U4 pad 14: (no net) -> unconnected-(U4-Q8-Pad14)
- U4 pad 15: (no net) -> unconnected-(U4-Q10-Pad15)
- U4 pad 2: (no net) -> unconnected-(U4-Q13-Pad2)
- U4 pad 4: (no net) -> unconnected-(U4-Q6-Pad4)
- U4 pad 5: (no net) -> unconnected-(U4-Q5-Pad5)
- U4 pad 6: (no net) -> unconnected-(U4-Q7-Pad6)
- U4 pad 7: (no net) -> unconnected-(U4-Q4-Pad7)
- U5 pad 5: (no net) -> unconnected-(U5-PG-Pad5)

Commit message: PSU re-layout: cables can be fitted, LM317s tab-down, isolated H2/H4
The audit against the PSU box found the board could not be wired:
- J1's wire entry faced the fuse clips 5 mm away; the mains gland sat in
  front of the IRM-05. J1 now faces the mains gland across a 17 mm
  parts-free bay (a no-footprint rule area).
- J2's mating face was 6 mm from the box wall, too close for the plug.
  It now looks at the output gland across a 24 mm free channel.
- H2/H4 standoffs (on PE) sat on the receiver GND pour behind only the
  solder mask: 5 mm copper keep-outs on both layers now.
- The clip-on heatsinks had no reserved space: the LM317s lie tab-down
  on copper areas of their OUT nets (stitched, both layers), no heatsinks.
- The MOV sits across the IRM-05's AC pins and the mains is hand-routed
  so unfused L and N never cross; tools/mains_clearance.py checks every
  mains gap (all >= 2.5 mm, >= 8 mm to the buckets and receiver side).
  J1 uses an elara variant with 2.3 mm pads (2.78 mm pin-to-pin creepage;
  the stock pads leave 2.48 mm).
- SRF1260 order code corrected to -102M.

Generated fit-check 3D models (tools/models3d.py -> PCB/elara.3dshapes)
for the parts KiCad has none for; kicadgen swaps them in on placement.
DRC 0 / unconnected 0 / parity 0.

Co-Authored-By: Claude Opus 5.5 <noreply@anthropic.com>
Claude-Session: https://claude.ai/code/session_01RsM1DhHhY1tSr2aHjVygSC
Parts:
- J1: footprint TerminalBlock_Phoenix:TerminalBlock_Phoenix_MKDS-1,5-3-5.08_1x03_P5.08mm_Horizontal -> elara:TerminalBlock_Phoenix_MKDS-1,5-3-5.08_1x03_P5.08mm_Horizontal_Mains
- U1, U2: footprint Package_TO_SOT_THT:TO-220-3_Vertical -> Package_TO_SOT_THT:TO-220-3_Horizontal_TabDown
- moved R4 28.3 mm to (120.5, 79.5), turned to 0 degrees
- moved R3 25.9 mm to (124.5, 79.5), turned to 0 degrees
- moved C3 24.9 mm to (128.5, 79.5), turned to 0 degrees
- moved U2 23.4 mm to (122.0, 75.0)
- moved C5 23.2 mm to (91.0, 76.5)
- moved R5 23.2 mm to (95.0, 76.5)
- moved D2 22.9 mm to (98.5, 76.5)
- moved D1 22.4 mm to (135.0, 66.0)
- moved RV1 21.5 mm to (79.0, 109.7), turned to 180 degrees
- moved C2 21.2 mm to (90.5, 64.0), turned to 0 degrees
- moved C4 20.9 mm to (87.5, 76.5)
- moved F1 20.8 mm to (85.0, 130.0), turned to 90 degrees
- moved R2 20.7 mm to (110.5, 79.5)
- moved R10 19.7 mm to (140.0, 66.0)
- moved U3 19.3 mm to (92.0, 70.5)
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Routing:
- net /Two-bucket isolated supply/COIL_N: track 74.4 -> 40.3 mm
- net GND_C: track 213.1 -> 186.0 mm, vias 59 -> 53
- net /Two-bucket isolated supply/AC_N: track 48.9 -> 25.7 mm
- net /Two-bucket isolated supply/AC_L: track 39.8 -> 19.5 mm
- net /Two-bucket isolated supply/L_IN: track 15.8 -> 33.0 mm
- net +12V_C: track 108.1 -> 124.2 mm, vias 2 -> 4
- net PE: track 107.6 -> 119.2 mm
- net /Two-bucket isolated supply/OSC_C: track 12.8 -> 4.65 mm, vias 2 -> 0
- net +15V_C: track 84.2 -> 76.3 mm, vias 2 -> 1
- net /Two-bucket isolated supply/OSC_X: track 19.7 -> 11.8 mm
- net /Two-bucket isolated supply/CHG_B: track 34.1 -> 42.0 mm
- net /Two-bucket isolated supply/CC_OUT: track 36.5 -> 31.7 mm
- net /Two-bucket isolated supply/CV_ADJ: track 18.3 -> 13.6 mm, vias 0 -> 1
- net +9V_OUT: track 34.4 -> 29.7 mm
- net /Two-bucket isolated supply/CC_SET: track 9.53 -> 5.80 mm, vias 0 -> 6
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- added copper zone on B.Cu, net /Two-bucket isolated supply/CC_SET
- added copper zone on F.Cu, net /Two-bucket isolated supply/CC_SET
- added copper zone on B.Cu, net /Two-bucket isolated supply/CHG
- added copper zone on F.Cu, net /Two-bucket isolated supply/CHG

Commit message: Mechanics on the real boards: fit check, PE stud, glands, docs and BOM
The mechanical models used invented placeholder parts, and the "clash
check" only compared whole units, so nothing inside the shield or the
PSU box was ever checked. Now:
- board_parts.py imports the populated boards from KiCad's STEP export
  (every part by reference); amp_pcb/psu_box use them, plus envelopes of
  the mated plugs and cable ends.
- fit_check.py checks every part and plug against every bar, lid, tray,
  screw, gland, standoff and the PE stud, the connector-to-wall gaps and
  the feed-through axis. It found the Micro-Fit's PCB-lock peg sitting on
  the tray rim: Ø5 x 3.5 relief pocket. All clear now; build_all runs it.
- Feed-through moved 4 mm onto the J201 axis. PSU glands in line with J1
  and J2 (mains low, output high); PE stud through the mains-end bar above
  the IRM-05 (it was under the board); nylon standoffs at H2/H4.
- Notches: AES3 16 x 13 for the pluggable header, BNC 16 x 14.
- 3D models: generated models are written as single products so KiCad
  names each instance by reference; radial cans and EDLCs get real-height
  models by MPN; C16 on its real 12.5 mm footprint (C17 moved).
- Exported assembly STEPs use part envelopes (the detailed boards are in
  PCB/*/fab); renders use the real parts.
- BOM: B6252HB BNC, Phoenix MC header + plug, 63 V WIMA, SRF1260-102M,
  no heatsinks, nylon standoffs, M4x20 PE screw. 516 EUR as designed, 411
  EUR recommended. Docs (ASSEMBLY, MOUNTING, MAINS_CABLE, STATUS,
  mechanical README, ORDERING, CLAUDE.md) follow the changes.

Co-Authored-By: Claude Opus 5.5 <noreply@anthropic.com>
Claude-Session: https://claude.ai/code/session_01RsM1DhHhY1tSr2aHjVygSC
Parts:
- C16: footprint Capacitor_THT:CP_Radial_D10.0mm_P5.00mm -> Capacitor_THT:CP_Radial_D12.5mm_P5.00mm
- moved C17 2.50 mm to (181.0, 130.5)
Routing:
- net /Two-bucket isolated supply/SET: track 40.4 -> 17.5 mm
- net GND: track 117.2 -> 126.5 mm, vias 63 -> 62
- net /Two-bucket isolated supply/LOAD_P: track 56.9 -> 59.3 mm

Commit message: Battery-friendly amplifier, RJ45 AES3 output, tidy placement, 1 mm PSU barrier
Amplifier schematic:
- No LEDs (battery use): the D301 overflow LED becomes test point TP301.
- PCM1804 FMT/S-M/OSR pins use the chip's internal 51 k pull-downs (6 resistors
  gone); BYPAS and the CS8406 mode pins get 47 k: about 3 mA less on +3V3.
- One output: AES3 on a shielded RJ45 (Amphenol RJHSE-5380, blue pair 4/5) for
  shielded twisted-pair cable, transformer isolated; the cable shield floats at
  the receiver (10 nF RF bond DNP, the DC bond is gone). The S/PDIF coax branch
  (BNC, second S22083, 5.6 mA standing current) is removed.

Layout:
- Amplifier re-placed in functional blocks on a 0.5 mm grid: PCM1804 and CS8406
  side by side so the I2S lines run straight, capacitor cells round the LDOs,
  DIP pull-downs in line with the switch pins, guard column in signal order with
  a re-routed hand guard-drive link. RJ45 notch 20 x 16 mm, BNC notch gone.
- PSU tidied (aligned columns, flyback diodes over their relays) and the charger
  / receiver copper kept >= 1.0 mm apart (was 0.30 mm): custom DRC rule, 1 mm
  router class for the relay contacts, hand-routed GND / GND_C at the relays.
- Reference labels follow each part's row; every label on silk except on the
  bare guard island. Fixed two placer bugs: each label counted as its own
  obstacle (SWIG proxies compared with 'is'), and unplaced labels blocked their
  neighbours. Texts are measured by their strokes, not KiCad's text cell.

Mechanics: RJ45 notch, plug envelope and a 1 mm isolation gap in fit_check.
BOM: 502 EUR as designed, 407 EUR recommended; 81 order lines.
Docs: STATUS, PLAN, ASSEMBLY, MOUNTING, README, mechanical and BOM notes;
MAINS_CABLE gains a certified DIY screened-cable option (H07RN-F + foil + braid)
and says why Ethernet cable must not carry mains.

All checks pass (tools/check_all.sh): ERC 0, DRC/parity 0 on all boards (only
the intended guard-island mask bridges), mains clearances, fit check, 27 tests.

Co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
Parts:
- moved C17 21.0 mm to (176.5, 110.0)
- moved R22 14.8 mm to (187.5, 112.5)
- moved C18 14.2 mm to (190.5, 112.5)
- moved D3 8.25 mm to (132.0, 93.5)
- moved D4 5.10 mm to (149.0, 93.5)
- moved R13 3.20 mm to (163.0, 110.0), turned to 90 degrees
- moved C19 3.04 mm to (187.5, 107.0)
- moved Q1 3.00 mm to (151.0, 87.0)
- moved R12 1.12 mm to (163.0, 101.5)
- moved C16 1.00 mm to (172.5, 121.0)
- moved C2 0.75 mm to (91.2, 64.0)
- moved U3 0.75 mm to (91.2, 70.5)
- moved R8 0.50 mm to (147.0, 82.5), turned to 90 degrees
Routing:
- net /Two-bucket isolated supply/LOAD_A: track 38.3 -> 83.7 mm, vias 0 -> 2
- net /Two-bucket isolated supply/VREG: track 40.0 -> 26.8 mm
- net /Two-bucket isolated supply/SET: track 17.5 -> 7.59 mm, vias 2 -> 0
- net /Two-bucket isolated supply/CC_OUT: track 31.7 -> 23.1 mm, vias 0 -> 1
- net /Two-bucket isolated supply/LOAD_P: track 59.3 -> 52.1 mm
- net /Two-bucket isolated supply/B_P: track 50.4 -> 57.3 mm
- net /Two-bucket isolated supply/LOAD_B: track 19.8 -> 26.5 mm, vias 0 -> 2
- net GND_C: track 186.0 -> 191.8 mm, vias 53 -> 56
- net /Two-bucket isolated supply/A_N: track 26.7 -> 32.3 mm
- net +15V_C: track 76.3 -> 72.1 mm, vias 1 -> 2
- net GND: track 126.5 -> 122.4 mm, vias 62 -> 59
- net /Two-bucket isolated supply/COIL_N: track 40.3 -> 36.5 mm
- net +12V_C: track 124.2 -> 120.9 mm, vias 4 -> 5
- net /Two-bucket isolated supply/GATE: track 8.63 -> 11.8 mm
- net /Two-bucket isolated supply/CV_ADJ: track 13.6 -> 16.3 mm, vias 1 -> 2
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