File: PCB/acdc_converter/acdc_converter.kicad_pcb (KiCad board)
At the start: 2 copper layers, 150 x 90 mm, 64 parts, among them J1 MAINS L N PE, J2 9V OUT, K1 G6K-2F-Y DC12, K2 G6K-2F-Y DC12, Q1 2N7002, U1 LM317, U2 LM317, U3 L78L12, U4 CD4060B, U5 LT3045

Commit message: AES3 source resistors 22 ohm for a 111 ohm source; tidy schematics and assembly drawings
- R412/R413 2 x 39 -> 2 x 22 ohm (Vishay TNPW060322R0BEEA, anti-sulfur): the
  CS8406 drivers are 33.5 ohm each at VL = 3.3 V, so 2 x 39 gave a 145 ohm
  source, outside AES3's 110 ohm +-20 %. The schematic note had used the 5 V
  figure and mis-added it.
- AES3 sheet: transformer flipped (kicadgen gains mirror='x') and wired straight
  to R412/R413/C405 and the RJ45, no more touching AES_HOT/AES_COLD labels.
- Stale S/PDIF and 9 V wording out of the sheets and BOM: DC input block reads
  6.98-15 V, J101 'DC IN', PSU J2 'DC OUT', reset button and clock branch say
  AES3; the legacy +9V / +9V_OUT net names are explained on the sheets.
- PSU root sheet gets the same power-path / board summary as the amplifier.
- Assembly drawings: fab-layer copies of the references removed wherever the
  silk reference shows (KiCad 9 texts cannot be hidden), so each part is named
  once; J201/J202 (no silk on the guard island) get theirs beside the part.
- BOM totals +0.14 EUR (502.15 ex VAT reference build, 407.22 recommended).

Co-Authored-By: Claude Opus 5.5 <noreply@anthropic.com>
Claude-Session: https://claude.ai/code/session_01RsM1DhHhY1tSr2aHjVygSC
Parts:
- J2: value 9V OUT -> DC OUT

Commit message: PSU charger at 10.4 V so the 2.7 V cells stay in rating; charger model corrected
The LM317 CV divider (240 R / 1.87 k) set 11.08 V, not the 10.9 V it was
labelled with: 2.72 V per EDLC cell whenever the receiver draws nothing,
2.83 V at the LM317's limits. R4 is now 1.74 k (10.4 V, 2.55 V per cell,
2.70 V worst case). Board copper and placement are unchanged; only R4's
value, the BOM and the order lists change.

The PSU model's charger now drops 6.2 ohm x I in the CC stage below 0.2 A
instead of a fixed 1.25 V. Re-run: 1.81 V of LT3045 headroom nominal,
1.05 V with every corner stacked. A 30 s swap is added as an option case
(0.36 V stacked), which replaces STATUS's unbacked claim that it drops out.
Also: the amplifier's +9V bus is about 6.0 V from the PSU (not 6.6 V),
and the PSU README's circuit line, CMC loop and margin figures are fixed.

Co-Authored-By: Claude Opus 5.5 <noreply@anthropic.com>
Claude-Session: https://claude.ai/code/session_01RsM1DhHhY1tSr2aHjVygSC
Parts:
- R4: value 1.87k -> 1.74k
