File: PCB/acdc_converter/psu.kicad_sch (KiCad schematic)
At the start: 64 parts, among them J1 MAINS L N PE, J2 9V OUT, K1 G6K-2F-Y DC12, K2 G6K-2F-Y DC12, Q1 2N7002, U1 LM317, U2 LM317, U3 L78L12, U4 CD4060B, U5 LT3045

Commit message: Route the two-bucket PSU board: fully connected, DRC clean but one thermal
Freerouting 1.9 in batch mode (2.1 never saved its session). Grounds
are routed on this board because the relays switch bucket current in
the unpoured area; mains nets 1.0 mm / 2.0 mm, current paths 0.6 mm;
hand-routed 1 mm PE rail on the left edge, GND_C-PE bond at the PE
hole; only the two mains-side holes are PE, the receiver-side holes
are unplated. Plain exposed-pad footprints (the thermal-via variants
need 0.2 mm drills). Newava S2208x redrawn as a 4-pin part (windings
1-2 / 3-4 per the DCR spec) with slotted pins 2/4 fitting either pitch.

Co-Authored-By: Claude Opus 5.5 <noreply@anthropic.com>
Claude-Session: https://claude.ai/code/session_01RsM1DhHhY1tSr2aHjVygSC
Parts:
- H2, H4: value M3 PE -> M3; footprint MountingHole:MountingHole_3.2mm_M3_Pad_Via -> MountingHole:MountingHole_3.2mm_M3; symbol Mechanical:MountingHole_Pad -> Mechanical:MountingHole
- U5: footprint Package_SO:MSOP-12-1EP_3x4.039mm_P0.65mm_EP1.651x2.845mm_ThermalVias -> Package_SO:MSOP-12-1EP_3x4.039mm_P0.65mm_EP1.651x2.845mm
Connections:
- net PE: no longer H2.1, H4.1
Other:
- moved on the sheet: H3

Commit message: Apply simulation fixes; add PSU/stability/system sims and priced BOM
simulations/psu: the charger caps each bucket at ~10.3 V, so the LT3045
at 8.45 V dropped out. Now R_SET 69.8k (6.98 V) and a 15 s swap
(CD4060 Rt 80.6k): +1.97 V headroom nominal, +0.49 V worst corner.
Charger output cap 10 uF -> 100 nF (3 A cold-start contact spike).
Swap artefact >= 83 dB below the floor; 50 Hz leakage 4-5 orders lower
than a direct AC-DC module (earth the receiver ground locally).
simulations/stability: guard buffer U202 had 43 deg worst-case phase
margin -> new C205 220 pF C0G GUARD-GND (56 deg). Others pass.
simulations/system: chain matches SPICE (45.8 nV/rtHz at SR1), ADC
transparent, 21 mV rms 50 Hz clip level; J202 = 100 G recommended with
an insulated antenna (10 G if bare).
bom/: priced BOM ~516 EUR ex VAT, ~406 EUR with the recommended
cost-down set; details and part checks in bom/README.md. Both
transformers are now S22083 (S22082 not stocked anywhere).
Layout: GND fan-out before routing, hand-routed guard drive, DIP
supply buses, NPTH pour keep-outs.

Co-Authored-By: Claude Opus 5.5 <noreply@anthropic.com>
Claude-Session: https://claude.ai/code/session_01RsM1DhHhY1tSr2aHjVygSC
Parts:
- C3: value 10u -> 100n; footprint Capacitor_SMD:C_1206_3216Metric -> Capacitor_SMD:C_0805_2012Metric; MPN GRM31CR71E106KA12L -> GRM21BR71H104KA01L
- R22: value 84.5k -> 69.8k; MPN ERA-6AEB8452V -> ERA-6AEB6982V
- R6: value 160k -> 80.6k; MPN ERA-6AEB164V -> ERA-6AEB8062V
Other:
- note added: "Buckets top out at ~10.3 V (two LM317 drops + SS34). 15 s at ~0.11 A droops ~0.7 V; LT3045 at 6.98 V keeps >= 0.5 V headroom in the worst corner (simulations/psu). Swap rate 33 mHz, below the ELF band."
- note added: "RECEIVER SIDE LT3045 6.98 V"
- note added: "SWAP TIMER Q14 toggles every ~15 s"
- note removed: "Bucket: 2.5 F feeding ~0.11 A for 30 s droops ~1.3 V (10.6 -> 9.3 V); LT3045 needs 8.45 + 0.3 V. Swap rate 17 mHz, below the ELF band."
- note removed: "RECEIVER SIDE LT3045 8.45 V"
- note removed: "SWAP TIMER Q14 toggles every ~30 s"
Changed lines of the file:
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@@
 			)
 		)
-		(property "Value" "10u"
+		(property "Value" "100n"
 			(at 287.31 72.72 0)
 			(effects
@@
 			)
 		)
-		(property "Footprint" "Capacitor_SMD:C_1206_3216Metric"
+		(property "Footprint" "Capacitor_SMD:C_0805_2012Metric"
 			(at 284.48 71.12 0)
 			(effects
@@
 			)
 		)
-		(property "Description" "MLCC 10u 25V X7R 1206"
+		(property "Description" "MLCC 100n 50V X7R 0805"
 			(at 284.48 71.12 0)
 			(effects
@@
 			)
 		)
-		(property "MPN" "GRM31CR71E106KA12L"
+		(property "MPN" "GRM21BR71H104KA01L"
 			(at 284.48 71.12 0)
 			(effects
@@
 			)
 		)
-		(property "Description" "14-stage counter + RC oscillator, f = 1/(2.3 Rt Ct) = 272 Hz, Q14 = f/16384"
+		(property "Description" "14-stage counter + RC oscillator, f = 1/(2.3 Rt Ct) = 540 Hz, Q14 toggles every ~15 s"
 			(at 55.88 147.32 0)
 			(effects
@@
 			)
 		)
-		(property "Value" "160k"
+		(property "Value" "80.6k"
 			(at 111.76 143.22 90)
 			(effects
@@
 			)
 		)
-		(property "Description" "Thin film 160k 0.1% 0805"
+		(property "Description" "Thin film 80.6k 0.1% 0805"
 			(at 111.76 139.7 0)
 			(effects
@@
 			)
 		)
-		(property "MPN" "ERA-6AEB164V"
+		(property "MPN" "ERA-6AEB8062V"
 			(at 111.76 139.7 0)
 			(effects
@@
 			)
 		)
-		(property "Value" "84.5k"
+		(property "Value" "69.8k"
 			(at 184.7 265.76 0)
 			(effects
@@
 			)
 		)
-		(property "Description" "Thin film 84.5k 0.1% 0805"
+		(property "Description" "Thin film 69.8k 0.1% 0805"
 			(at 182.88 264.16 0)
 			(effects
@@
 			)
 		)
-		(property "MPN" "ERA-6AEB8452V"
+		(property "MPN" "ERA-6AEB6982V"
 			(at 182.88 264.16 0)
 			(effects
@@
 			)
 		)
-		(property "Description" "Micro-Fit 3.0 2-pin, 8.45 V to the antenna amplifier (shielded pair)"
+		(property "Description" "Micro-Fit 3.0 2-pin, 6.98 V to the antenna amplifier (shielded pair)"
 			(at 274.32 241.3 0)
 			(effects
@@
 		)
 	)
-	(text "SWAP TIMER  Q14 toggles every ~30 s"
+	(text "SWAP TIMER  Q14 toggles every ~15 s"
 		(exclude_from_sim no)
 		(at 16.27 108.2 0)
@@
 		)
 	)
-	(text "RECEIVER SIDE  LT3045 8.45 V"
+	(text "RECEIVER SIDE  LT3045 6.98 V"
 		(exclude_from_sim no)
 		(at 130.27 203.2 0)
@@
 		)
 	)
-	(text "Bucket: 2.5 F feeding ~0.11 A for 30 s droops ~1.3 V (10.6 -> 9.3 V); LT3045 needs 8.45 + 0.3 V. Swap rate 17 mHz, below the ELF band."
+	(text "Buckets top out at ~10.3 V (two LM317 drops + SS34). 15 s at ~0.11 A droops ~0.7 V; LT3045 at 6.98 V keeps >= 0.5 V headroom in the worst corner (simulations/psu). Swap rate 33 mHz, below the ELF band."
 		(exclude_from_sim no)
 		(at 15 290 0)

Commit message: EDLC cells: HV1030-2R7106-R (10 x 30 mm) in the PSU design; BOM totals refreshed (518 / 408 EUR)
Co-Authored-By: Claude Opus 5.5 <noreply@anthropic.com>
Claude-Session: https://claude.ai/code/session_01RsM1DhHhY1tSr2aHjVygSC
Parts:
- C10, C11, C12, C13, C14, C15, C8, C9: MPN HV1245-2R7106-R -> HV1030-2R7106-R
Changed lines of the file:
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@@
 			)
 		)
-		(property "Description" "EDLC 10 F 2.7 V, D12.5 P5.0 (any 10 F 2.7 V radial cell; match within 5%)"
+		(property "Description" "EDLC 10 F 2.7 V, D10 x 30 mm, P5.0 (any 10 F 2.7 V radial cell; match within 5%)"
 			(at 30.48 226.06 0)
 			(effects
@@
 			)
 		)
-		(property "MPN" "HV1245-2R7106-R"
+		(property "MPN" "HV1030-2R7106-R"
 			(at 30.48 226.06 0)
 			(effects
@@
 			)
 		)
-		(property "Description" "EDLC 10 F 2.7 V, D12.5 P5.0 (any 10 F 2.7 V radial cell; match within 5%)"
+		(property "Description" "EDLC 10 F 2.7 V, D10 x 30 mm, P5.0 (any 10 F 2.7 V radial cell; match within 5%)"
 			(at 30.48 233.68 0)
 			(effects
@@
 			)
 		)
-		(property "MPN" "HV1245-2R7106-R"
+		(property "MPN" "HV1030-2R7106-R"
 			(at 30.48 233.68 0)
 			(effects
@@
 			)
 		)
-		(property "Description" "EDLC 10 F 2.7 V, D12.5 P5.0 (any 10 F 2.7 V radial cell; match within 5%)"
+		(property "Description" "EDLC 10 F 2.7 V, D10 x 30 mm, P5.0 (any 10 F 2.7 V radial cell; match within 5%)"
 			(at 30.48 241.3 0)
 			(effects
@@
 			)
 		)
-		(property "MPN" "HV1245-2R7106-R"
+		(property "MPN" "HV1030-2R7106-R"
 			(at 30.48 241.3 0)
 			(effects
@@
 			)
 		)
-		(property "Description" "EDLC 10 F 2.7 V, D12.5 P5.0 (any 10 F 2.7 V radial cell; match within 5%)"
+		(property "Description" "EDLC 10 F 2.7 V, D10 x 30 mm, P5.0 (any 10 F 2.7 V radial cell; match within 5%)"
 			(at 30.48 248.92 0)
 			(effects
@@
 			)
 		)
-		(property "MPN" "HV1245-2R7106-R"
+		(property "MPN" "HV1030-2R7106-R"
 			(at 30.48 248.92 0)
 			(effects
@@
 			)
 		)
-		(property "Description" "EDLC 10 F 2.7 V, D12.5 P5.0 (any 10 F 2.7 V radial cell; match within 5%)"
+		(property "Description" "EDLC 10 F 2.7 V, D10 x 30 mm, P5.0 (any 10 F 2.7 V radial cell; match within 5%)"
 			(at 87.63 226.06 0)
 			(effects
@@
 			)
 		)
-		(property "MPN" "HV1245-2R7106-R"
+		(property "MPN" "HV1030-2R7106-R"
 			(at 87.63 226.06 0)
 			(effects
@@
 			)
 		)
-		(property "Description" "EDLC 10 F 2.7 V, D12.5 P5.0 (any 10 F 2.7 V radial cell; match within 5%)"
+		(property "Description" "EDLC 10 F 2.7 V, D10 x 30 mm, P5.0 (any 10 F 2.7 V radial cell; match within 5%)"
 			(at 87.63 233.68 0)
 			(effects
@@
 			)
 		)
-		(property "MPN" "HV1245-2R7106-R"
+		(property "MPN" "HV1030-2R7106-R"
 			(at 87.63 233.68 0)
 			(effects
@@
 			)
 		)
-		(property "Description" "EDLC 10 F 2.7 V, D12.5 P5.0 (any 10 F 2.7 V radial cell; match within 5%)"
+		(property "Description" "EDLC 10 F 2.7 V, D10 x 30 mm, P5.0 (any 10 F 2.7 V radial cell; match within 5%)"
 			(at 87.63 241.3 0)
 			(effects
@@
 			)
 		)
-		(property "MPN" "HV1245-2R7106-R"
+		(property "MPN" "HV1030-2R7106-R"
 			(at 87.63 241.3 0)
 			(effects
@@
 			)
 		)
-		(property "Description" "EDLC 10 F 2.7 V, D12.5 P5.0 (any 10 F 2.7 V radial cell; match within 5%)"
+		(property "Description" "EDLC 10 F 2.7 V, D10 x 30 mm, P5.0 (any 10 F 2.7 V radial cell; match within 5%)"
 			(at 87.63 248.92 0)
 			(effects
@@
 			)
 		)
-		(property "MPN" "HV1245-2R7106-R"
+		(property "MPN" "HV1030-2R7106-R"
 			(at 87.63 248.92 0)
 			(effects

Commit message: Pedantic DRC/ERC pass: schematic parity clean, BNC notch, island without silk
- Board nets carry the schematic's names (sheet-path prefix on local nets, KiCad's
  unconnected-(...) nets on open pins): DRC schematic parity 0 on both boards.
- BNC: its mounting lugs reached 1.4 mm under the right-hand wall, whose round
  barrel hole left the bar resting on them (tilted wall, BNC shell = S/PDIF return
  shorted to the shield). The frame now has a 16 x 14 mm notch there, and the
  strip copper stops clear of the lugs. Micro-Fit notch widened to 14 mm.
- Guard island: mask opening follows the island outline; LMP7721 and the bias link
  use project footprint variants without silk on the island (no ink on the
  femtoamp surface). tools/fp_variants.py derives them from the stock footprints.
- S22083 footprint: silk outline no longer crosses its own slotted pads.
- CS8406 as a project symbol with pin 1 typed as the hardware-mode COPY/C input:
  ERC 0 on both schematics. PSU mounting holes out of the BOM; plate and PSU
  projects register the elara footprint library.
- Remaining amplifier DRC items: 79 solder-mask-bridge warnings, all on the
  deliberately unmasked guard island. PSU and plate boards: 0 of anything.

Co-Authored-By: Claude Opus 5.5 <noreply@anthropic.com>
Claude-Session: https://claude.ai/code/session_01RsM1DhHhY1tSr2aHjVygSC
Parts:
- H1, H2, H3, H4: now left out of the parts list
Changed lines of the file:
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@@
 		(unit 1)
 		(exclude_from_sim no)
-		(in_bom yes)
+		(in_bom no)
 		(on_board yes)
 		(dnp no)
@@
 		(unit 1)
 		(exclude_from_sim no)
-		(in_bom yes)
+		(in_bom no)
 		(on_board yes)
 		(dnp no)
@@
 		(unit 1)
 		(exclude_from_sim no)
-		(in_bom yes)
+		(in_bom no)
 		(on_board yes)
 		(dnp no)
@@
 		(unit 1)
 		(exclude_from_sim no)
-		(in_bom yes)
-		(on_board yes)
-		(dnp no)
+		(in_bom no)
+		(on_board yes)
+		(dnp no)

Commit message: Pedantic schematic and silkscreen pass: zero overlaps, labels clear of tracks
Schematics
- tools/kicadgen/schcheck.py checks KiCad's own SVG rendering (exact stroke boxes)
  for text over text, lines through text, crowded twin labels and text outside the
  frame. Both schematics: 0 findings; ERC 0 on both.
- Generator: Sheet.join (one wire + one label instead of two facing labels),
  per-symbol field positions, per-pin stub lengths, shared power symbol for
  adjacent top/bottom rail pins, crowded rail runs get one label, longer PCM1804
  pins (no-connect cross clear of the pin number), PE value clear of its symbol.
- Fixed: doubled VIN_RAW/BIAS_DIV/LED_OVF/CV_ADJ/LED_C labels, +5VA vs VREG,
  +5V_PRE twins, CS8406 GND straps vs neighbours, BNC/LED/diode fields over their
  graphics, bucket-cell values vs tap labels, notes outside the frame, J2 -> J202.
- Root sheet: sub-sheets in signal-flow order with arrows and a design summary;
  dated title blocks.

Boards
- References prefer spots clear of tracks as well as parts (two candidate rings);
  compartment labels are re-placed after routing; the title block on the back is
  placed as one unit; no stitching via under any board text.
- DRC with schematic parity: amplifier 0 errors / 0 unconnected / 0 parity (only
  the intended bare-island mask warnings); PSU and plate 0 of anything.

Co-Authored-By: Claude Opus 5.5 <noreply@anthropic.com>
Claude-Session: https://claude.ai/code/session_01RsM1DhHhY1tSr2aHjVygSC
Other:
- note added: "15 s at ~0.11 A droops ~0.7 V; the LT3045 at 6.98 V keeps"
- note added: ">= 0.5 V headroom in the worst corner (simulations/psu)."
- note added: "Buckets top out at ~10.3 V (two LM317 drops + SS34)."
- note added: "Swap rate 33 mHz, far below the ELF band."
- note removed: "Buckets top out at ~10.3 V (two LM317 drops + SS34). 15 s at ~0.11 A droops ~0.7 V; LT3045 at 6.98 V keeps >= 0.5 V headroom in the worst corner (simulations/psu). Swap rate 33 mHz, below the ELF band."
- moved on the sheet: C1, C17, C2, D3, D4, J1, R1

Commit message: PSU re-layout: cables can be fitted, LM317s tab-down, isolated H2/H4
The audit against the PSU box found the board could not be wired:
- J1's wire entry faced the fuse clips 5 mm away; the mains gland sat in
  front of the IRM-05. J1 now faces the mains gland across a 17 mm
  parts-free bay (a no-footprint rule area).
- J2's mating face was 6 mm from the box wall, too close for the plug.
  It now looks at the output gland across a 24 mm free channel.
- H2/H4 standoffs (on PE) sat on the receiver GND pour behind only the
  solder mask: 5 mm copper keep-outs on both layers now.
- The clip-on heatsinks had no reserved space: the LM317s lie tab-down
  on copper areas of their OUT nets (stitched, both layers), no heatsinks.
- The MOV sits across the IRM-05's AC pins and the mains is hand-routed
  so unfused L and N never cross; tools/mains_clearance.py checks every
  mains gap (all >= 2.5 mm, >= 8 mm to the buckets and receiver side).
  J1 uses an elara variant with 2.3 mm pads (2.78 mm pin-to-pin creepage;
  the stock pads leave 2.48 mm).
- SRF1260 order code corrected to -102M.

Generated fit-check 3D models (tools/models3d.py -> PCB/elara.3dshapes)
for the parts KiCad has none for; kicadgen swaps them in on placement.
DRC 0 / unconnected 0 / parity 0.

Co-Authored-By: Claude Opus 5.5 <noreply@anthropic.com>
Claude-Session: https://claude.ai/code/session_01RsM1DhHhY1tSr2aHjVygSC
Parts:
- J1: footprint TerminalBlock_Phoenix:TerminalBlock_Phoenix_MKDS-1,5-3-5.08_1x03_P5.08mm_Horizontal -> elara:TerminalBlock_Phoenix_MKDS-1,5-3-5.08_1x03_P5.08mm_Horizontal_Mains
- L1: MPN SRF1260-102Y -> SRF1260-102M
- U1, U2: footprint Package_TO_SOT_THT:TO-220-3_Vertical -> Package_TO_SOT_THT:TO-220-3_Horizontal_TabDown
Changed lines of the file:
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@@
 			)
 		)
-		(property "Footprint" "TerminalBlock_Phoenix:TerminalBlock_Phoenix_MKDS-1,5-3-5.08_1x03_P5.08mm_Horizontal"
+		(property "Footprint" "elara:TerminalBlock_Phoenix_MKDS-1,5-3-5.08_1x03_P5.08mm_Horizontal_Mains"
 			(at 33.02 45.72 0)
 			(effects
@@
 			)
 		)
-		(property "Description" "Mains input: 1 L, 2 N, 3 PE"
+		(property "Description" "Mains input: 1 L, 2 N, 3 PE (2.3 mm pads: 2.78 mm creepage pin to pin)"
 			(at 33.02 45.72 0)
 			(effects
@@
 			)
 		)
-		(property "Footprint" "Package_TO_SOT_THT:TO-220-3_Vertical"
+		(property "Footprint" "Package_TO_SOT_THT:TO-220-3_Horizontal_TabDown"
 			(at 210.82 38.1 0)
 			(effects
@@
 			)
 		)
-		(property "Description" "Constant current, 1.25 V / 6.2 R = 0.2 A (clip-on heatsink)"
+		(property "Description" "Constant current, 1.25 V / 6.2 R = 0.2 A (tab = OUT = CC_SET, bolted to a copper area)"
 			(at 210.82 38.1 0)
 			(effects
@@
 			)
 		)
-		(property "Footprint" "Package_TO_SOT_THT:TO-220-3_Vertical"
+		(property "Footprint" "Package_TO_SOT_THT:TO-220-3_Horizontal_TabDown"
 			(at 251.46 38.1 0)
 			(effects
@@
 			)
 		)
-		(property "Description" "Constant voltage 1.25 V x (1 + 1.87k/240) = 10.9 V"
+		(property "Description" "Constant voltage 1.25 V x (1 + 1.87k/240) = 10.9 V (tab bolted to a CHG copper area)"
 			(at 251.46 38.1 0)
 			(effects
@@
 			)
 		)
-		(property "MPN" "SRF1260-102Y"
+		(property "MPN" "SRF1260-102M"
 			(at 241.3 223.52 0)
 			(effects

Commit message: Mechanics on the real boards: fit check, PE stud, glands, docs and BOM
The mechanical models used invented placeholder parts, and the "clash
check" only compared whole units, so nothing inside the shield or the
PSU box was ever checked. Now:
- board_parts.py imports the populated boards from KiCad's STEP export
  (every part by reference); amp_pcb/psu_box use them, plus envelopes of
  the mated plugs and cable ends.
- fit_check.py checks every part and plug against every bar, lid, tray,
  screw, gland, standoff and the PE stud, the connector-to-wall gaps and
  the feed-through axis. It found the Micro-Fit's PCB-lock peg sitting on
  the tray rim: Ø5 x 3.5 relief pocket. All clear now; build_all runs it.
- Feed-through moved 4 mm onto the J201 axis. PSU glands in line with J1
  and J2 (mains low, output high); PE stud through the mains-end bar above
  the IRM-05 (it was under the board); nylon standoffs at H2/H4.
- Notches: AES3 16 x 13 for the pluggable header, BNC 16 x 14.
- 3D models: generated models are written as single products so KiCad
  names each instance by reference; radial cans and EDLCs get real-height
  models by MPN; C16 on its real 12.5 mm footprint (C17 moved).
- Exported assembly STEPs use part envelopes (the detailed boards are in
  PCB/*/fab); renders use the real parts.
- BOM: B6252HB BNC, Phoenix MC header + plug, 63 V WIMA, SRF1260-102M,
  no heatsinks, nylon standoffs, M4x20 PE screw. 516 EUR as designed, 411
  EUR recommended. Docs (ASSEMBLY, MOUNTING, MAINS_CABLE, STATUS,
  mechanical README, ORDERING, CLAUDE.md) follow the changes.

Co-Authored-By: Claude Opus 5.5 <noreply@anthropic.com>
Claude-Session: https://claude.ai/code/session_01RsM1DhHhY1tSr2aHjVygSC
Parts:
- C16: footprint Capacitor_THT:CP_Radial_D10.0mm_P5.00mm -> Capacitor_THT:CP_Radial_D12.5mm_P5.00mm
Changed lines of the file:
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@@
 			)
 		)
-		(property "Footprint" "Capacitor_THT:CP_Radial_D10.0mm_P5.00mm"
+		(property "Footprint" "Capacitor_THT:CP_Radial_D12.5mm_P5.00mm"
 			(at 139.7 243.84 0)
 			(effects
@@
 			)
 		)
-		(property "Description" "Electrolytic 2200u 16V low-ESR, rides through the relay transit"
+		(property "Description" "Electrolytic 2200u 16V low-ESR, 12.5 x 20 mm, rides through the relay transit"
 			(at 139.7 243.84 0)
 			(effects
