File: PCB/acdc_converter/psu.kicad_sch (KiCad schematic)
At the start: 64 parts, among them J1 MAINS L N PE, J2 DC OUT, K1 G6K-2F-Y DC12, K2 G6K-2F-Y DC12, Q1 2N7002, U1 LM317, U2 LM317, U3 L78L12, U4 CD4060B, U5 LT3045

Commit message: PSU charger at 10.4 V so the 2.7 V cells stay in rating; charger model corrected
The LM317 CV divider (240 R / 1.87 k) set 11.08 V, not the 10.9 V it was
labelled with: 2.72 V per EDLC cell whenever the receiver draws nothing,
2.83 V at the LM317's limits. R4 is now 1.74 k (10.4 V, 2.55 V per cell,
2.70 V worst case). Board copper and placement are unchanged; only R4's
value, the BOM and the order lists change.

The PSU model's charger now drops 6.2 ohm x I in the CC stage below 0.2 A
instead of a fixed 1.25 V. Re-run: 1.81 V of LT3045 headroom nominal,
1.05 V with every corner stacked. A 30 s swap is added as an option case
(0.36 V stacked), which replaces STATUS's unbacked claim that it drops out.
Also: the amplifier's +9V bus is about 6.0 V from the PSU (not 6.6 V),
and the PSU README's circuit line, CMC loop and margin figures are fixed.

Co-Authored-By: Claude Opus 5.5 <noreply@anthropic.com>
Claude-Session: https://claude.ai/code/session_01RsM1DhHhY1tSr2aHjVygSC
Parts:
- R4: value 1.87k -> 1.74k; MPN ERA-6AEB1871V -> ERA-6AEB1741V
Other:
- note added: "15 s at ~0.1 A droops ~0.6 V; the LT3045 at 6.98 V keeps"
- note added: ">= 1 V headroom in the worst corner (simulations/psu)."
- note added: "Buckets swing 9.4-10.1 V (CV 10.4 V: 2.6 V per cell)."
- note added: "CHARGER (GND_C) CC 0.2 A -> CV 10.4 V"
- note removed: "15 s at ~0.11 A droops ~0.7 V; the LT3045 at 6.98 V keeps"
- note removed: ">= 0.5 V headroom in the worst corner (simulations/psu)."
- note removed: "Buckets top out at ~10.3 V (two LM317 drops + SS34)."
- note removed: "CHARGER (GND_C) CC 0.2 A -> CV 10.9 V"
Changed lines of the file:
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@@
 			)
 		)
-		(property "Description" "Constant voltage 1.25 V x (1 + 1.87k/240) = 10.9 V (tab bolted to a CHG copper area)"
+		(property "Description" "Constant voltage 1.25 V x (1 + 1.74k/240) + 50 uA x 1.74k = 10.4 V, cells <= 2.7 V at the LM317 limits (tab bolted to a CHG copper area)"
 			(at 251.46 38.1 0)
 			(effects
@@
 			)
 		)
-		(property "Value" "1.87k"
+		(property "Value" "1.74k"
 			(at 273.6 85.42 0)
 			(effects
@@
 			)
 		)
-		(property "Description" "Thin film 1.87k 0.1% 0805"
+		(property "Description" "Thin film 1.74k 0.1% 0805"
 			(at 271.78 83.82 0)
 			(effects
@@
 			)
 		)
-		(property "MPN" "ERA-6AEB1871V"
+		(property "MPN" "ERA-6AEB1741V"
 			(at 271.78 83.82 0)
 			(effects
@@
 		)
 	)
-	(text "CHARGER  (GND_C)  CC 0.2 A -> CV 10.9 V"
+	(text "CHARGER  (GND_C)  CC 0.2 A -> CV 10.4 V"
 		(exclude_from_sim no)
 		(at 171.27 23.2 0)
@@
 		)
 	)
-	(text "Buckets top out at ~10.3 V (two LM317 drops + SS34)."
+	(text "Buckets swing 9.4-10.1 V (CV 10.4 V: 2.6 V per cell)."
 		(exclude_from_sim no)
 		(at 290 212 0)
@@
 		)
 	)
-	(text "15 s at ~0.11 A droops ~0.7 V; the LT3045 at 6.98 V keeps"
+	(text "15 s at ~0.1 A droops ~0.6 V; the LT3045 at 6.98 V keeps"
 		(exclude_from_sim no)
 		(at 290 217 0)
@@
 		)
 	)
-	(text ">= 0.5 V headroom in the worst corner (simulations/psu)."
+	(text ">= 1 V headroom in the worst corner (simulations/psu)."
 		(exclude_from_sim no)
 		(at 290 222 0)
