File: PCB/plate_capacitor/plate_capacitor.kicad_pcb (KiCad board)
At the start: 2 copper layers, 64 x 64 mm, 5 parts, among them J1 PLATE

Commit message: Title blocks (rev 0.2) on all boards; PSU starved thermal fixed (C4 ground pad solid) -- PSU DRC fully clean
Fab packages regenerated for all three boards.

Co-Authored-By: Claude Opus 5.5 <noreply@anthropic.com>
Claude-Session: https://claude.ai/code/session_01RsM1DhHhY1tSr2aHjVygSC
Parts:
- NP1, NP2, NP3, NP4: footprint (none) -> elara:Hole_NPTH

Commit message: Plate capacitors: solder tongues outside the gap; fab packages refreshed
The plate had its only plated solder hole inside the 64 x 64 square, so
the fillet and lead end on the copper face sat 0.5 mm from the facing
plate. The mechanical model meanwhile assumed side pads fed by vias,
which matched neither. Now every plate has two 7 x 8 mm tongues (left
edge 20 mm, right edge 44 mm from the top); a plate turned over
left-right puts its tongues where the other has none, so each joint is
outside the overlap. Node plates use both tongues, GND plates one. The
CadQuery model, wiring and resistor runs follow the real tongues.
C unchanged: 48.9 pF bare, 51.9 pF masked. DRC 0.

Fab packages for all three boards regenerated (Gerbers, drill, pos, BOM,
PDFs, render, STEP with the board corner as origin, interactive BOM).

Co-Authored-By: Claude Opus 5.5 <noreply@anthropic.com>
Claude-Session: https://claude.ai/code/session_01RsM1DhHhY1tSr2aHjVygSC
Parts:
- added J2: PLATE, , F.Cu at (117.5, 94.0)
- moved J1 47.3 mm to (46.5, 70.0)
Other:
- board size 64 x 64 mm -> 78 x 64 mm
- board text added: "PAIR: TURN ONE PLATE OVER LEFT-RIGHT, TONGUES APART"
- board text added: "SOLDER ON THE TONGUES ONLY"
- board text removed: "PAIR: FLIP ONE PLATE, TABS MUST NOT OVERLAP"
- board text removed: "SOLDER THE TAB FROM THIS SIDE ONLY"
